File: CleanLVSupply/CleanLVSupply/5v.kicad_sch (KiCad schematic)
At the start: 19 parts, among them U5 LMR54406F, U6 TPS7A47

Commit message: CleanLVSupply routing progress
Parts:
- renumbered C32 to C31, C30 to C32, C31 to C33, C33 to C34, C34 to C35, C35 to C36, C40 to C39, C41 to C40, C36 to C41, C39 to C42
Changed lines of the file:
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@@
 		(dnp no)
 		(fields_autoplaced yes)
-		(property "Reference" "C35"
+		(property "Reference" "C36"
 			(at 204.47 69.8499 0)
 			(effects
@@
 			(project "CleanLVSupply"
 				(path "/4327ef59-ef76-48f2-90b1-1a9e4399cfc2/bede3db6-f65b-4911-9741-402d7e0e6982"
-					(reference "C35")
+					(reference "C36")
 					(unit 1)
 				)
@@
 		(dnp no)
 		(fields_autoplaced yes)
-		(property "Reference" "C34"
+		(property "Reference" "C35"
 			(at 186.69 69.8499 0)
 			(effects
@@
 			(project "CleanLVSupply"
 				(path "/4327ef59-ef76-48f2-90b1-1a9e4399cfc2/bede3db6-f65b-4911-9741-402d7e0e6982"
-					(reference "C34")
+					(reference "C35")
 					(unit 1)
 				)
@@
 		(dnp no)
 		(fields_autoplaced yes)
-		(property "Reference" "C40"
+		(property "Reference" "C39"
 			(at 186.69 123.1899 0)
 			(effects
@@
 			(project "CleanLVSupply"
 				(path "/4327ef59-ef76-48f2-90b1-1a9e4399cfc2/bede3db6-f65b-4911-9741-402d7e0e6982"
-					(reference "C40")
+					(reference "C39")
 					(unit 1)
 				)
@@
 		(dnp no)
 		(fields_autoplaced yes)
-		(property "Reference" "C30"
+		(property "Reference" "C32"
 			(at 77.47 69.8499 0)
 			(effects
@@
 			(project "CleanLVSupply"
 				(path "/4327ef59-ef76-48f2-90b1-1a9e4399cfc2/bede3db6-f65b-4911-9741-402d7e0e6982"
-					(reference "C30")
+					(reference "C32")
 					(unit 1)
 				)
@@
 		(dnp no)
 		(fields_autoplaced yes)
-		(property "Reference" "C36"
+		(property "Reference" "C41"
 			(at 88.9 129.9209 0)
 			(effects
@@
 			(project "CleanLVSupply"
 				(path "/4327ef59-ef76-48f2-90b1-1a9e4399cfc2/bede3db6-f65b-4911-9741-402d7e0e6982"
-					(reference "C36")
+					(reference "C41")
 					(unit 1)
 				)
@@
 		(dnp no)
 		(fields_autoplaced yes)
-		(property "Reference" "C33"
+		(property "Reference" "C34"
 			(at 173.99 69.8499 0)
 			(effects
@@
 			(project "CleanLVSupply"
 				(path "/4327ef59-ef76-48f2-90b1-1a9e4399cfc2/bede3db6-f65b-4911-9741-402d7e0e6982"
-					(reference "C33")
+					(reference "C34")
 					(unit 1)
 				)
@@
 		(dnp no)
 		(fields_autoplaced yes)
-		(property "Reference" "C39"
+		(property "Reference" "C42"
 			(at 135.89 130.8099 0)
 			(effects
@@
 			(project "CleanLVSupply"
 				(path "/4327ef59-ef76-48f2-90b1-1a9e4399cfc2/bede3db6-f65b-4911-9741-402d7e0e6982"
-					(reference "C39")
+					(reference "C42")
 					(unit 1)
 				)
@@
 		(dnp no)
 		(fields_autoplaced yes)
-		(property "Reference" "C41"
+		(property "Reference" "C40"
 			(at 204.47 122.3009 0)
 			(effects
@@
 			(project "CleanLVSupply"
 				(path "/4327ef59-ef76-48f2-90b1-1a9e4399cfc2/bede3db6-f65b-4911-9741-402d7e0e6982"
-					(reference "C41")
+					(reference "C40")
 					(unit 1)
 				)
@@
 		(dnp no)
 		(fields_autoplaced yes)
-		(property "Reference" "C31"
+		(property "Reference" "C33"
 			(at 95.25 69.8499 0)
 			(effects
@@
 			(project "CleanLVSupply"
 				(path "/4327ef59-ef76-48f2-90b1-1a9e4399cfc2/bede3db6-f65b-4911-9741-402d7e0e6982"
-					(reference "C31")
+					(reference "C33")
 					(unit 1)
 				)
@@
 		(dnp no)
 		(fields_autoplaced yes)
-		(property "Reference" "C32"
+		(property "Reference" "C31"
 			(at 132.0863 57.15 90)
 			(effects
@@
 			(project "CleanLVSupply"
 				(path "/4327ef59-ef76-48f2-90b1-1a9e4399cfc2/bede3db6-f65b-4911-9741-402d7e0e6982"
-					(reference "C32")
-					(unit 1)
-				)
+					(reference "C31")
+					(unit 1)
+				)
