File: CleanLVSupply/CleanLVSupply/m15v.kicad_sch (KiCad schematic)
At the start: 31 parts, among them U1 LM25576, U2 TPS7A30

Commit message: CleanLVSupply routing progress
Parts:
- renumbered C5 to C10, C6 to C11, C9 to C12, C15 to C13, C13 to C15, C12 to C16, C16 to C19, C7 to C2, C1 to C3, C2 to C4, C3 to C5, C10 to C6, C11 to C7, C4 to C9, R3 to R1, R1 to R2, R5 to R3, R2 to R4, R4 to R5, R8 to R6, R6 to R7, R7 to R8
Changed lines of the file:
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@@
 		(dnp no)
 		(fields_autoplaced yes)
-		(property "Reference" "R8"
+		(property "Reference" "R6"
 			(at 172.72 126.9999 0)
 			(effects
@@
 			(project "CleanLVSupply"
 				(path "/4327ef59-ef76-48f2-90b1-1a9e4399cfc2/1251894f-ff7f-4119-a254-b437dbce5fd5"
-					(reference "R8")
+					(reference "R6")
 					(unit 1)
 				)
@@
 		(dnp no)
 		(fields_autoplaced yes)
-		(property "Reference" "C11"
+		(property "Reference" "C7"
 			(at 251.46 66.4209 0)
 			(effects
@@
 			(project ""
 				(path "/4327ef59-ef76-48f2-90b1-1a9e4399cfc2/1251894f-ff7f-4119-a254-b437dbce5fd5"
-					(reference "C11")
+					(reference "C7")
 					(unit 1)
 				)
@@
 		(dnp no)
 		(fields_autoplaced yes)
-		(property "Reference" "R1"
+		(property "Reference" "R2"
 			(at 113.03 64.7699 0)
 			(effects
@@
 			(project "CleanLVSupply"
 				(path "/4327ef59-ef76-48f2-90b1-1a9e4399cfc2/1251894f-ff7f-4119-a254-b437dbce5fd5"
-					(reference "R1")
+					(reference "R2")
 					(unit 1)
 				)
@@
 		(dnp no)
 		(fields_autoplaced yes)
-		(property "Reference" "C15"
+		(property "Reference" "C13"
 			(at 123.19 124.4599 0)
 			(effects
@@
 			(project "CleanLVSupply"
 				(path "/4327ef59-ef76-48f2-90b1-1a9e4399cfc2/1251894f-ff7f-4119-a254-b437dbce5fd5"
-					(reference "C15")
+					(reference "C13")
 					(unit 1)
 				)
@@
 		(on_board yes)
 		(dnp no)
-		(property "Reference" "C9"
+		(property "Reference" "C12"
 			(at 185.42 82.042 90)
 			(effects
@@
 			(project "CleanLVSupply"
 				(path "/4327ef59-ef76-48f2-90b1-1a9e4399cfc2/1251894f-ff7f-4119-a254-b437dbce5fd5"
-					(reference "C9")
+					(reference "C12")
 					(unit 1)
 				)
@@
 		(dnp no)
 		(fields_autoplaced yes)
-		(property "Reference" "C4"
+		(property "Reference" "C9"
 			(at 97.79 77.4699 0)
 			(effects
@@
 			(project "CleanLVSupply"
 				(path "/4327ef59-ef76-48f2-90b1-1a9e4399cfc2/1251894f-ff7f-4119-a254-b437dbce5fd5"
-					(reference "C4")
+					(reference "C9")
 					(unit 1)
 				)
@@
 		(dnp no)
 		(fields_autoplaced yes)
-		(property "Reference" "C5"
+		(property "Reference" "C10"
 			(at 114.3 77.4699 0)
 			(effects
@@
 			(project "CleanLVSupply"
 				(path "/4327ef59-ef76-48f2-90b1-1a9e4399cfc2/1251894f-ff7f-4119-a254-b437dbce5fd5"
-					(reference "C5")
+					(reference "C10")
 					(unit 1)
 				)
@@
 		(dnp no)
 		(fields_autoplaced yes)
-		(property "Reference" "R5"
+		(property "Reference" "R3"
 			(at 190.5 67.31 90)
 			(effects
@@
 			(project "CleanLVSupply"
 				(path "/4327ef59-ef76-48f2-90b1-1a9e4399cfc2/1251894f-ff7f-4119-a254-b437dbce5fd5"
-					(reference "R5")
+					(reference "R3")
 					(unit 1)
 				)
@@
 		(dnp no)
 		(fields_autoplaced yes)
-		(property "Reference" "C13"
+		(property "Reference" "C15"
 			(at 87.63 133.3499 0)
 			(effects
@@
 			(project "CleanLVSupply"
 				(path "/4327ef59-ef76-48f2-90b1-1a9e4399cfc2/1251894f-ff7f-4119-a254-b437dbce5fd5"
-					(reference "C13")
+					(reference "C15")
 					(unit 1)
 				)
@@
 		(dnp no)
 		(fields_autoplaced yes)
-		(property "Reference" "R2"
+		(property "Reference" "R4"
 			(at 127 77.4699 0)
 			(effects
@@
 			(project "CleanLVSupply"
 				(path "/4327ef59-ef76-48f2-90b1-1a9e4399cfc2/1251894f-ff7f-4119-a254-b437dbce5fd5"
-					(reference "R2")
+					(reference "R4")
 					(unit 1)
 				)
@@
 		(dnp no)
 		(fields_autoplaced yes)
-		(property "Reference" "R7"
+		(property "Reference" "R8"
 			(at 172.72 139.6999 0)
 			(effects
@@
 			(project "CleanLVSupply"
 				(path "/4327ef59-ef76-48f2-90b1-1a9e4399cfc2/1251894f-ff7f-4119-a254-b437dbce5fd5"
-					(reference "R7")
+					(reference "R8")
 					(unit 1)
 				)
@@
 		(dnp no)
 		(fields_autoplaced yes)
-		(property "Reference" "C2"
+		(property "Reference" "C4"
 			(at 66.04 57.1499 0)
 			(effects
@@
 			(project "CleanLVSupply"
 				(path "/4327ef59-ef76-48f2-90b1-1a9e4399cfc2/1251894f-ff7f-4119-a254-b437dbce5fd5"
-					(reference "C2")
+					(reference "C4")
 					(unit 1)
 				)
@@
 		(dnp no)
 		(fields_autoplaced yes)
-		(property "Reference" "C1"
+		(property "Reference" "C3"
 			(at 48.26 57.1499 0)
 			(effects
@@
 			(project ""
 				(path "/4327ef59-ef76-48f2-90b1-1a9e4399cfc2/1251894f-ff7f-4119-a254-b437dbce5fd5"
-					(reference "C1")
+					(reference "C3")
 					(unit 1)
 				)
@@
 		(dnp no)
 		(fields_autoplaced yes)
-		(property "Reference" "C16"
+		(property "Reference" "C19"
 			(at 162.56 139.6999 0)
 			(effects
@@
 			(project "CleanLVSupply"
 				(path "/4327ef59-ef76-48f2-90b1-1a9e4399cfc2/1251894f-ff7f-4119-a254-b437dbce5fd5"
-					(reference "C16")
+					(reference "C19")
 					(unit 1)
 				)
@@
 		(dnp no)
 		(fields_autoplaced yes)
-		(property "Reference" "R3"
+		(property "Reference" "R1"
 			(at 219.71 55.8799 0)
 			(effects
@@
 			(project "CleanLVSupply"
 				(path "/4327ef59-ef76-48f2-90b1-1a9e4399cfc2/1251894f-ff7f-4119-a254-b437dbce5fd5"
-					(reference "R3")
+					(reference "R1")
 					(unit 1)
 				)
@@
 		(dnp no)
 		(fields_autoplaced yes)
-		(property "Reference" "C3"
+		(property "Reference" "C5"
 			(at 83.82 67.3099 0)
 			(effects
@@
 			(project "CleanLVSupply"
 				(path "/4327ef59-ef76-48f2-90b1-1a9e4399cfc2/1251894f-ff7f-4119-a254-b437dbce5fd5"
-					(reference "C3")
+					(reference "C5")
 					(unit 1)
 				)
@@
 		(dnp no)
 		(fields_autoplaced yes)
-		(property "Reference" "R6"
+		(property "Reference" "R7"
 			(at 69.85 139.6999 0)
 			(effects
@@
 			(project "CleanLVSupply"
 				(path "/4327ef59-ef76-48f2-90b1-1a9e4399cfc2/1251894f-ff7f-4119-a254-b437dbce5fd5"
-					(reference "R6")
+					(reference "R7")
 					(unit 1)
 				)
@@
 		(dnp no)
 		(fields_autoplaced yes)
-		(property "Reference" "R4"
+		(property "Reference" "R5"
 			(at 219.71 77.4699 0)
 			(effects
@@
 			(project "CleanLVSupply"
 				(path "/4327ef59-ef76-48f2-90b1-1a9e4399cfc2/1251894f-ff7f-4119-a254-b437dbce5fd5"
-					(reference "R4")
+					(reference "R5")
 					(unit 1)
 				)
@@
 		(dnp no)
 		(fields_autoplaced yes)
-		(property "Reference" "C6"
+		(property "Reference" "C11"
 			(at 142.24 77.4699 0)
 			(effects
@@
 			(project "CleanLVSupply"
 				(path "/4327ef59-ef76-48f2-90b1-1a9e4399cfc2/1251894f-ff7f-4119-a254-b437dbce5fd5"
-					(reference "C6")
+					(reference "C11")
 					(unit 1)
 				)
@@
 		(dnp no)
 		(fields_autoplaced yes)
-		(property "Reference" "C10"
+		(property "Reference" "C6"
 			(at 234.95 67.3099 0)
 			(effects
@@
 			(project "CleanLVSupply"
 				(path "/4327ef59-ef76-48f2-90b1-1a9e4399cfc2/1251894f-ff7f-4119-a254-b437dbce5fd5"
-					(reference "C10")
+					(reference "C6")
 					(unit 1)
 				)
@@
 		(dnp no)
 		(fields_autoplaced yes)
-		(property "Reference" "C7"
+		(property "Reference" "C2"
 			(at 177.8063 43.18 90)
 			(effects
@@
 			(project ""
 				(path "/4327ef59-ef76-48f2-90b1-1a9e4399cfc2/1251894f-ff7f-4119-a254-b437dbce5fd5"
-					(reference "C7")
+					(reference "C2")
 					(unit 1)
 				)
@@
 		(dnp no)
 		(fields_autoplaced yes)
-		(property "Reference" "C12"
+		(property "Reference" "C16"
 			(at 105.41 133.3499 0)
 			(effects
@@
 			(project "CleanLVSupply"
 				(path "/4327ef59-ef76-48f2-90b1-1a9e4399cfc2/1251894f-ff7f-4119-a254-b437dbce5fd5"
-					(reference "C12")
-					(unit 1)
-				)
+					(reference "C16")
+					(unit 1)
+				)
