File: HiFiDAC/diff-amp.kicad_sch (KiCad schematic)
At the start: 11 parts, among them U7 OPA1612

Commit message: HiFiDAC renumbered and footprints assigned
Parts:
- C40: renamed from C25; footprint (none) -> BW_PassiveMechanical:C_0704_1810Metric
- C41: renamed from C26; footprint (none) -> BW_PassiveMechanical:C_0704_1810Metric
- R43: renamed from R24; footprint (none) -> Resistor_SMD:R_0805_2012Metric
- R44: renamed from R23; footprint (none) -> Resistor_SMD:R_0805_2012Metric
- R45: renamed from R25; footprint (none) -> Resistor_SMD:R_0805_2012Metric
- R46: renamed from R26; footprint (none) -> Resistor_SMD:R_0805_2012Metric
- R47: renamed from R27; footprint (none) -> Resistor_SMD:R_0805_2012Metric
- R48: renamed from R28; footprint (none) -> Resistor_SMD:R_0805_2012Metric
- R49: renamed from R29; footprint (none) -> Resistor_SMD:R_0805_2012Metric
- R50: renamed from R30; footprint (none) -> Resistor_SMD:R_0805_2012Metric
- U7: footprint (none) -> Package_SON:WSON-8-1EP_3x3mm_P0.5mm_EP1.2x2mm
Changed lines of the file:
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@@
 		(dnp no)
 		(fields_autoplaced yes)
-		(property "Reference" "#PWR020"
+		(property "Reference" "#PWR040"
 			(at 209.55 80.01 0)
 			(effects
@@
 			(project "HiFiDAC"
 				(path "/9ca5e549-4577-422c-b8f3-d4e6ad408ec3/ee079862-ea8e-4560-9a6a-6f0a2816074e"
-					(reference "#PWR020")
+					(reference "#PWR040")
 					(unit 1)
 				)
@@
 		(dnp no)
 		(fields_autoplaced yes)
-		(property "Reference" "#PWR021"
+		(property "Reference" "#PWR043"
 			(at 209.55 100.33 0)
 			(effects
@@
 			(project "HiFiDAC"
 				(path "/9ca5e549-4577-422c-b8f3-d4e6ad408ec3/ee079862-ea8e-4560-9a6a-6f0a2816074e"
-					(reference "#PWR021")
+					(reference "#PWR043")
 					(unit 1)
 				)
@@
 		(dnp no)
 		(fields_autoplaced yes)
-		(property "Reference" "R29"
+		(property "Reference" "R49"
 			(at 85.09 132.08 90)
 			(effects
@@
 			)
 		)
-		(property "Footprint" ""
+		(property "Footprint" "Resistor_SMD:R_0805_2012Metric"
 			(at 84.836 139.446 90)
 			(effects
@@
 			(project "HiFiDAC"
 				(path "/9ca5e549-4577-422c-b8f3-d4e6ad408ec3/ee079862-ea8e-4560-9a6a-6f0a2816074e"
-					(reference "R29")
+					(reference "R49")
 					(unit 1)
 				)
@@
 		(dnp no)
 		(fields_autoplaced yes)
-		(property "Reference" "R30"
+		(property "Reference" "R50"
 			(at 96.52 143.5099 0)
 			(effects
@@
 			)
 		)
-		(property "Footprint" ""
+		(property "Footprint" "Resistor_SMD:R_0805_2012Metric"
 			(at 94.996 145.034 90)
 			(effects
@@
 			(project "HiFiDAC"
 				(path "/9ca5e549-4577-422c-b8f3-d4e6ad408ec3/ee079862-ea8e-4560-9a6a-6f0a2816074e"
-					(reference "R30")
+					(reference "R50")
 					(unit 1)
 				)
@@
 		(dnp no)
 		(fields_autoplaced yes)
-		(property "Reference" "R27"
+		(property "Reference" "R47"
 			(at 107.95 111.76 90)
 			(effects
@@
 			)
 		)
-		(property "Footprint" ""
+		(property "Footprint" "Resistor_SMD:R_0805_2012Metric"
 			(at 107.696 119.126 90)
 			(effects
@@
 			(project "HiFiDAC"
 				(path "/9ca5e549-4577-422c-b8f3-d4e6ad408ec3/ee079862-ea8e-4560-9a6a-6f0a2816074e"
-					(reference "R27")
+					(reference "R47")
 					(unit 1)
 				)
@@
 		(dnp no)
 		(fields_autoplaced yes)
-		(property "Reference" "#PWR019"
+		(property "Reference" "#PWR044"
 			(at 93.98 157.48 0)
 			(effects
@@
 			(project "HiFiDAC"
 				(path "/9ca5e549-4577-422c-b8f3-d4e6ad408ec3/ee079862-ea8e-4560-9a6a-6f0a2816074e"
-					(reference "#PWR019")
+					(reference "#PWR044")
 					(unit 1)
 				)
@@
 		(dnp no)
 		(fields_autoplaced yes)
-		(property "Reference" "#PWR018"
+		(property "Reference" "#PWR042"
 			(at 93.98 100.33 0)
 			(effects
@@
 			(project "HiFiDAC"
 				(path "/9ca5e549-4577-422c-b8f3-d4e6ad408ec3/ee079862-ea8e-4560-9a6a-6f0a2816074e"
-					(reference "#PWR018")
+					(reference "#PWR042")
 					(unit 1)
 				)
@@
 		(dnp no)
 		(fields_autoplaced yes)
-		(property "Reference" "R24"
+		(property "Reference" "R43"
 			(at 107.95 54.61 90)
 			(effects
@@
 			)
 		)
-		(property "Footprint" ""
+		(property "Footprint" "Resistor_SMD:R_0805_2012Metric"
 			(at 107.696 61.976 90)
 			(effects
@@
 			(project "HiFiDAC"
 				(path "/9ca5e549-4577-422c-b8f3-d4e6ad408ec3/ee079862-ea8e-4560-9a6a-6f0a2816074e"
-					(reference "R24")
+					(reference "R43")
 					(unit 1)
 				)
@@
 		(dnp no)
 		(fields_autoplaced yes)
-		(property "Reference" "R26"
+		(property "Reference" "R46"
 			(at 96.52 86.3599 0)
 			(effects
@@
 			)
 		)
-		(property "Footprint" ""
+		(property "Footprint" "Resistor_SMD:R_0805_2012Metric"
 			(at 94.996 87.884 90)
 			(effects
@@
 			(project "HiFiDAC"
 				(path "/9ca5e549-4577-422c-b8f3-d4e6ad408ec3/ee079862-ea8e-4560-9a6a-6f0a2816074e"
-					(reference "R26")
+					(reference "R46")
 					(unit 1)
 				)
@@
 			)
 		)
-		(property "Footprint" ""
+		(property "Footprint" "Package_SON:WSON-8-1EP_3x3mm_P0.5mm_EP1.2x2mm"
 			(at 106.68 133.35 0)
 			(effects
@@
 		(dnp no)
 		(fields_autoplaced yes)
-		(property "Reference" "R23"
+		(property "Reference" "R44"
 			(at 85.09 64.77 90)
 			(effects
@@
 			)
 		)
-		(property "Footprint" ""
+		(property "Footprint" "Resistor_SMD:R_0805_2012Metric"
 			(at 84.836 72.136 90)
 			(effects
@@
 			(project "HiFiDAC"
 				(path "/9ca5e549-4577-422c-b8f3-d4e6ad408ec3/ee079862-ea8e-4560-9a6a-6f0a2816074e"
-					(reference "R23")
+					(reference "R44")
 					(unit 1)
 				)
@@
 		(dnp no)
 		(fields_autoplaced yes)
-		(property "Reference" "#PWR017"
+		(property "Reference" "#PWR041"
 			(at 243.84 90.17 0)
 			(effects
@@
 			(project "HiFiDAC"
 				(path "/9ca5e549-4577-422c-b8f3-d4e6ad408ec3/ee079862-ea8e-4560-9a6a-6f0a2816074e"
-					(reference "#PWR017")
+					(reference "#PWR041")
 					(unit 1)
 				)
@@
 		(dnp no)
 		(fields_autoplaced yes)
-		(property "Reference" "R25"
+		(property "Reference" "R45"
 			(at 85.09 74.93 90)
 			(effects
@@
 			)
 		)
-		(property "Footprint" ""
+		(property "Footprint" "Resistor_SMD:R_0805_2012Metric"
 			(at 84.836 82.296 90)
 			(effects
@@
 			(project "HiFiDAC"
 				(path "/9ca5e549-4577-422c-b8f3-d4e6ad408ec3/ee079862-ea8e-4560-9a6a-6f0a2816074e"
-					(reference "R25")
+					(reference "R45")
 					(unit 1)
 				)
@@
 		(dnp no)
 		(fields_autoplaced yes)
-		(property "Reference" "R28"
+		(property "Reference" "R48"
 			(at 85.09 121.92 90)
 			(effects
@@
 			)
 		)
-		(property "Footprint" ""
+		(property "Footprint" "Resistor_SMD:R_0805_2012Metric"
 			(at 84.836 129.286 90)
 			(effects
@@
 			(project "HiFiDAC"
 				(path "/9ca5e549-4577-422c-b8f3-d4e6ad408ec3/ee079862-ea8e-4560-9a6a-6f0a2816074e"
-					(reference "R28")
+					(reference "R48")
 					(unit 1)
 				)
@@
 			)
 		)
-		(property "Footprint" ""
+		(property "Footprint" "Package_SON:WSON-8-1EP_3x3mm_P0.5mm_EP1.2x2mm"
 			(at 217.17 90.17 0)
 			(effects
@@
 		(dnp no)
 		(fields_autoplaced yes)
-		(property "Reference" "C25"
+		(property "Reference" "C40"
 			(at 236.22 83.8199 0)
 			(effects
@@
 			)
 		)
-		(property "Footprint" ""
+		(property "Footprint" "BW_PassiveMechanical:C_0704_1810Metric"
 			(at 231.4448 81.28 0)
 			(effects
@@
 			(project "HiFiDAC"
 				(path "/9ca5e549-4577-422c-b8f3-d4e6ad408ec3/ee079862-ea8e-4560-9a6a-6f0a2816074e"
-					(reference "C25")
+					(reference "C40")
 					(unit 1)
 				)
@@
 			)
 		)
-		(property "Footprint" ""
+		(property "Footprint" "Package_SON:WSON-8-1EP_3x3mm_P0.5mm_EP1.2x2mm"
 			(at 106.68 76.2 0)
 			(effects
@@
 		(dnp no)
 		(fields_autoplaced yes)
-		(property "Reference" "C26"
+		(property "Reference" "C41"
 			(at 236.22 93.9799 0)
 			(effects
@@
 			)
 		)
-		(property "Footprint" ""
+		(property "Footprint" "BW_PassiveMechanical:C_0704_1810Metric"
 			(at 231.4448 91.44 0)
 			(effects
@@
 			(project "HiFiDAC"
 				(path "/9ca5e549-4577-422c-b8f3-d4e6ad408ec3/ee079862-ea8e-4560-9a6a-6f0a2816074e"
-					(reference "C26")
-					(unit 1)
-				)
+					(reference "C41")
+					(unit 1)
+				)

Commit message: HiFiDAC PCB progress, slight shape changes
Connections:
- net VL_SE: now also U7.7; no longer U7.1
- net VR_SE: now also U7.1; no longer U7.7
- net at R49.1, R50.1: now also U7.3 (+); no longer U7.5 (+)
- net at R47.2, R48.1: now also U7.2 (-); no longer U7.6 (-)
- net at R43.2, R44.1: now also U7.6 (-); no longer U7.2 (-)
- net at R45.1, R46.1: now also U7.5 (+); no longer U7.3 (+)
Other:
- moved on the sheet: U7A, U7B

Commit message: HiFiDAC redesign of clocking, digital IO, ferrite beads
Parts:
- renumbered C40 to C43, C41 to C44, R43 to R37, R44 to R38, R45 to R39, R46 to R40, R47 to R41, R48 to R42, R49 to R43, R50 to R44, U7 to U8
Changed lines of the file:
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@@
 		(dnp no)
 		(fields_autoplaced yes)
-		(property "Reference" "#PWR040"
+		(property "Reference" "#PWR041"
 			(at 209.55 80.01 0)
 			(effects
@@
 			(project "HiFiDAC"
 				(path "/9ca5e549-4577-422c-b8f3-d4e6ad408ec3/ee079862-ea8e-4560-9a6a-6f0a2816074e"
-					(reference "#PWR040")
+					(reference "#PWR041")
 					(unit 1)
 				)
@@
 		(dnp no)
 		(fields_autoplaced yes)
-		(property "Reference" "#PWR043"
+		(property "Reference" "#PWR044"
 			(at 209.55 100.33 0)
 			(effects
@@
 			(project "HiFiDAC"
 				(path "/9ca5e549-4577-422c-b8f3-d4e6ad408ec3/ee079862-ea8e-4560-9a6a-6f0a2816074e"
-					(reference "#PWR043")
+					(reference "#PWR044")
 					(unit 1)
 				)
@@
 		(dnp no)
 		(fields_autoplaced yes)
-		(property "Reference" "R49"
+		(property "Reference" "R43"
 			(at 85.09 132.08 90)
 			(effects
@@
 			(project "HiFiDAC"
 				(path "/9ca5e549-4577-422c-b8f3-d4e6ad408ec3/ee079862-ea8e-4560-9a6a-6f0a2816074e"
-					(reference "R49")
+					(reference "R43")
 					(unit 1)
 				)
@@
 		(dnp no)
 		(fields_autoplaced yes)
-		(property "Reference" "R50"
+		(property "Reference" "R44"
 			(at 96.52 143.5099 0)
 			(effects
@@
 			(project "HiFiDAC"
 				(path "/9ca5e549-4577-422c-b8f3-d4e6ad408ec3/ee079862-ea8e-4560-9a6a-6f0a2816074e"
-					(reference "R50")
+					(reference "R44")
 					(unit 1)
 				)
@@
 		(dnp no)
 		(fields_autoplaced yes)
-		(property "Reference" "R47"
+		(property "Reference" "R41"
 			(at 107.95 111.76 90)
 			(effects
@@
 			(project "HiFiDAC"
 				(path "/9ca5e549-4577-422c-b8f3-d4e6ad408ec3/ee079862-ea8e-4560-9a6a-6f0a2816074e"
-					(reference "R47")
+					(reference "R41")
 					(unit 1)
 				)
@@
 		(dnp no)
 		(fields_autoplaced yes)
-		(property "Reference" "#PWR044"
+		(property "Reference" "#PWR045"
 			(at 93.98 157.48 0)
 			(effects
@@
 			(project "HiFiDAC"
 				(path "/9ca5e549-4577-422c-b8f3-d4e6ad408ec3/ee079862-ea8e-4560-9a6a-6f0a2816074e"
-					(reference "#PWR044")
+					(reference "#PWR045")
 					(unit 1)
 				)
@@
 		(dnp no)
 		(fields_autoplaced yes)
-		(property "Reference" "#PWR042"
+		(property "Reference" "#PWR043"
 			(at 93.98 100.33 0)
 			(effects
@@
 			(project "HiFiDAC"
 				(path "/9ca5e549-4577-422c-b8f3-d4e6ad408ec3/ee079862-ea8e-4560-9a6a-6f0a2816074e"
-					(reference "#PWR042")
+					(reference "#PWR043")
 					(unit 1)
 				)
@@
 		(dnp no)
 		(fields_autoplaced yes)
-		(property "Reference" "R43"
+		(property "Reference" "R37"
 			(at 107.95 54.61 90)
 			(effects
@@
 			(project "HiFiDAC"
 				(path "/9ca5e549-4577-422c-b8f3-d4e6ad408ec3/ee079862-ea8e-4560-9a6a-6f0a2816074e"
-					(reference "R43")
+					(reference "R37")
 					(unit 1)
 				)
@@
 		(dnp no)
 		(fields_autoplaced yes)
-		(property "Reference" "R46"
+		(property "Reference" "R40"
 			(at 96.52 86.3599 0)
 			(effects
@@
 			(project "HiFiDAC"
 				(path "/9ca5e549-4577-422c-b8f3-d4e6ad408ec3/ee079862-ea8e-4560-9a6a-6f0a2816074e"
-					(reference "R46")
+					(reference "R40")
 					(unit 1)
 				)
@@
 		(dnp no)
 		(fields_autoplaced yes)
-		(property "Reference" "U7"
+		(property "Reference" "U8"
 			(at 107.95 64.77 0)
 			(effects
@@
 			(project ""
 				(path "/9ca5e549-4577-422c-b8f3-d4e6ad408ec3/ee079862-ea8e-4560-9a6a-6f0a2816074e"
-					(reference "U7")
+					(reference "U8")
 					(unit 2)
 				)
@@
 		(dnp no)
 		(fields_autoplaced yes)
-		(property "Reference" "R44"
+		(property "Reference" "R38"
 			(at 85.09 64.77 90)
 			(effects
@@
 			(project "HiFiDAC"
 				(path "/9ca5e549-4577-422c-b8f3-d4e6ad408ec3/ee079862-ea8e-4560-9a6a-6f0a2816074e"
-					(reference "R44")
+					(reference "R38")
 					(unit 1)
 				)
@@
 		(dnp no)
 		(fields_autoplaced yes)
-		(property "Reference" "#PWR041"
+		(property "Reference" "#PWR042"
 			(at 243.84 90.17 0)
 			(effects
@@
 			(project "HiFiDAC"
 				(path "/9ca5e549-4577-422c-b8f3-d4e6ad408ec3/ee079862-ea8e-4560-9a6a-6f0a2816074e"
-					(reference "#PWR041")
+					(reference "#PWR042")
 					(unit 1)
 				)
@@
 		(dnp no)
 		(fields_autoplaced yes)
-		(property "Reference" "R45"
+		(property "Reference" "R39"
 			(at 85.09 74.93 90)
 			(effects
@@
 			(project "HiFiDAC"
 				(path "/9ca5e549-4577-422c-b8f3-d4e6ad408ec3/ee079862-ea8e-4560-9a6a-6f0a2816074e"
-					(reference "R45")
+					(reference "R39")
 					(unit 1)
 				)
@@
 		(dnp no)
 		(fields_autoplaced yes)
-		(property "Reference" "R48"
+		(property "Reference" "R42"
 			(at 85.09 121.92 90)
 			(effects
@@
 			(project "HiFiDAC"
 				(path "/9ca5e549-4577-422c-b8f3-d4e6ad408ec3/ee079862-ea8e-4560-9a6a-6f0a2816074e"
-					(reference "R48")
+					(reference "R42")
 					(unit 1)
 				)
@@
 		(dnp no)
 		(fields_autoplaced yes)
-		(property "Reference" "U7"
+		(property "Reference" "U8"
 			(at 220.98 88.8999 0)
 			(effects
@@
 			(project ""
 				(path "/9ca5e549-4577-422c-b8f3-d4e6ad408ec3/ee079862-ea8e-4560-9a6a-6f0a2816074e"
-					(reference "U7")
+					(reference "U8")
 					(unit 3)
 				)
@@
 		(dnp no)
 		(fields_autoplaced yes)
-		(property "Reference" "C40"
+		(property "Reference" "C43"
 			(at 236.22 83.8199 0)
 			(effects
@@
 			(project "HiFiDAC"
 				(path "/9ca5e549-4577-422c-b8f3-d4e6ad408ec3/ee079862-ea8e-4560-9a6a-6f0a2816074e"
-					(reference "C40")
+					(reference "C43")
 					(unit 1)
 				)
@@
 		(dnp no)
 		(fields_autoplaced yes)
-		(property "Reference" "U7"
+		(property "Reference" "U8"
 			(at 107.95 121.92 0)
 			(effects
@@
 			(project ""
 				(path "/9ca5e549-4577-422c-b8f3-d4e6ad408ec3/ee079862-ea8e-4560-9a6a-6f0a2816074e"
-					(reference "U7")
+					(reference "U8")
 					(unit 1)
 				)
@@
 		(dnp no)
 		(fields_autoplaced yes)
-		(property "Reference" "C41"
+		(property "Reference" "C44"
 			(at 236.22 93.9799 0)
 			(effects
@@
 			(project "HiFiDAC"
 				(path "/9ca5e549-4577-422c-b8f3-d4e6ad408ec3/ee079862-ea8e-4560-9a6a-6f0a2816074e"
-					(reference "C41")
-					(unit 1)
-				)
+					(reference "C44")
+					(unit 1)
+				)
