File: HiFiDAC/i-v-stage.kicad_sch (KiCad schematic)
At the start: 44 parts, among them U3 OPA1612, U4 OPA1612, U5 OPA1612, U6 OPA1612

Commit message: HiFiDAC renumbered and footprints assigned
Parts:
- C20: renamed from C5; footprint (none) -> Capacitor_SMD:C_0603_1608Metric
- C21: renamed from C7; footprint (none) -> Capacitor_SMD:C_0603_1608Metric
- C22: renamed from C6; footprint (none) -> Capacitor_SMD:C_0603_1608Metric
- C23: renamed from C17; footprint (none) -> BW_PassiveMechanical:C_0704_1810Metric
- C24: renamed from C19; footprint (none) -> BW_PassiveMechanical:C_0704_1810Metric
- C25: renamed from C8; footprint (none) -> Capacitor_SMD:C_0603_1608Metric
- C26: renamed from C10; footprint (none) -> Capacitor_SMD:C_0603_1608Metric
- C27: renamed from C18; footprint (none) -> BW_PassiveMechanical:C_0704_1810Metric
- C28: renamed from C20; footprint (none) -> BW_PassiveMechanical:C_0704_1810Metric
- C29: renamed from C9; footprint (none) -> Capacitor_SMD:C_0603_1608Metric
- C30: renamed from C21; footprint (none) -> BW_PassiveMechanical:C_0704_1810Metric
- C31: renamed from C23; footprint (none) -> BW_PassiveMechanical:C_0704_1810Metric
- C32: renamed from C22; footprint (none) -> BW_PassiveMechanical:C_0704_1810Metric
- C33: renamed from C24; footprint (none) -> BW_PassiveMechanical:C_0704_1810Metric
- C34: renamed from C11; footprint (none) -> Capacitor_SMD:C_0603_1608Metric
- C35: renamed from C12; footprint (none) -> Capacitor_SMD:C_0603_1608Metric
- C36: renamed from C13; footprint (none) -> Capacitor_SMD:C_0603_1608Metric
- C37: renamed from C14; footprint (none) -> Capacitor_SMD:C_0603_1608Metric
- C38: renamed from C15; footprint (none) -> Capacitor_SMD:C_0603_1608Metric
- C39: renamed from C16; footprint (none) -> Capacitor_SMD:C_0603_1608Metric
- R23: renamed from R3; footprint (none) -> Resistor_SMD:R_0805_2012Metric
- R24: renamed from R4; footprint (none) -> Resistor_SMD:R_0805_2012Metric
- R25: renamed from R7; footprint (none) -> Resistor_SMD:R_0805_2012Metric
- R26: renamed from R5; footprint (none) -> Resistor_SMD:R_0805_2012Metric
- R27: renamed from R6; footprint (none) -> Resistor_SMD:R_0805_2012Metric
- R28: renamed from R8; footprint (none) -> Resistor_SMD:R_0805_2012Metric
- R29: renamed from R9; footprint (none) -> Resistor_SMD:R_0805_2012Metric
- R30: renamed from R12; footprint (none) -> Resistor_SMD:R_0805_2012Metric
- R31: renamed from R10; footprint (none) -> Resistor_SMD:R_0805_2012Metric
- R32: renamed from R11; footprint (none) -> Resistor_SMD:R_0805_2012Metric
- R33: renamed from R13; footprint (none) -> Resistor_SMD:R_0805_2012Metric
- R34: renamed from R14; footprint (none) -> Resistor_SMD:R_0805_2012Metric
- R35: renamed from R15; footprint (none) -> Resistor_SMD:R_0805_2012Metric
- R36: renamed from R16; footprint (none) -> Resistor_SMD:R_0805_2012Metric
- R37: renamed from R17; footprint (none) -> Resistor_SMD:R_0805_2012Metric
- R38: renamed from R18; footprint (none) -> Resistor_SMD:R_0805_2012Metric
- R39: renamed from R19; footprint (none) -> Resistor_SMD:R_0805_2012Metric
- R40: renamed from R20; footprint (none) -> Resistor_SMD:R_0805_2012Metric
- R41: renamed from R21; footprint (none) -> Resistor_SMD:R_0805_2012Metric
- R42: renamed from R22; footprint (none) -> Resistor_SMD:R_0805_2012Metric
- U3, U4, U5, U6: footprint (none) -> Package_SON:WSON-8-1EP_3x3mm_P0.5mm_EP1.2x2mm

Commit message: HiFiDAC redesign of clocking, digital IO, ferrite beads
Parts:
- renumbered C20 to C23, C21 to C24, C22 to C25, C23 to C26, C24 to C27, C25 to C28, C26 to C29, C27 to C30, C28 to C31, C29 to C32, C30 to C33, C31 to C34, C32 to C35, C33 to C36, C34 to C37, C35 to C38, C36 to C39, C37 to C40, C38 to C41, C39 to C42, R23 to R17, R24 to R18, R25 to R19, R26 to R20, R27 to R21, R28 to R22, R29 to R23, R30 to R24, R31 to R25, R32 to R26, R33 to R27, R34 to R28, R35 to R29, R36 to R30, R37 to R31, R38 to R32, R39 to R33, R40 to R34, R41 to R35, R42 to R36, U3 to U4, U4 to U5, U5 to U6, U6 to U7

Commit message: HiFiDAC v2 progress
Parts:
- removed C37, C40: 2.2nF C0G, Capacitor_SMD:C_0603_1608Metric, symbol Device:C
- removed C38, C39, C41, C42: 2.7nF C0G, Capacitor_SMD:C_0603_1608Metric, symbol Device:C
- removed R33: 4.7kΩRS, Resistor_SMD:R_0805_2012Metric, symbol Device:R_US
- removed R34, R36: 330ΩRS, Resistor_SMD:R_0805_2012Metric, symbol Device:R_US
- removed R35: 470ΩRS, Resistor_SMD:R_0805_2012Metric, symbol Device:R_US
- removed U6, U7: OPA1612, Package_SON:WSON-8-1EP_3x3mm_P0.5mm_EP1.2x2mm, symbol BW_Active:OPA1612
- C23: value 2.2nF C0G -> 1nF C0G
- C24, C29: value 2.7nF C0G -> 1nF C0G
- C25, C32: value 2.7nF C0G -> 33pF C0G
- C27, C31, C34: value 0.1µF C0G -> 10nF C0G; footprint BW_PassiveMechanical:C_0704_1810Metric -> Capacitor_SMD:C_0603_1608Metric
- C28: value 2.2nF C0G -> 10nF C0G
- C36: value 0.1µF C0G -> 1nF C0G; footprint BW_PassiveMechanical:C_0704_1810Metric -> Capacitor_SMD:C_0603_1608Metric
- R17, R32: value 1kΩRS -> 22kΩRS
- R18: value 4.7kΩRS -> 3.3kΩRS
- R19: value 330ΩRS -> 22kΩRS
- R20: value 470ΩRS -> 3.3kΩRS
- R21, R29: value 330ΩRS -> 4.7kΩRS
- R22: value 1kΩRS -> 4.7kΩRS
- R23: value 4.7kΩRS -> 100ΩRS
- R24: value 330ΩRS -> 100ΩRS
- R25: value 470ΩRS -> 22kΩRS
- R26, R31: value 330ΩRS -> 3.3kΩRS
- R27: value 1kΩRS -> 100ΩRS
- R30: value 470ΩRS -> 100ΩRS
Connections:
- net +15V: no longer C27.2, C34.2
- net -15V: no longer C31.1, C36.1
- net GND: now also C28.1, C31.1; no longer C25.1, C31.2, C32.1, C36.2, R21.1, R26.1, R31.1, U4.5 (+), U5.5 (+)
- net IL+: now also C23.1, R17.1, R18.1, U4.5 (+); no longer C28.1, R22.1, R23.1, U4.6 (-)
- net IL-: now also C24.1, R19.1, R20.1, U4.6 (-); no longer C23.1, R17.1, R18.1, U4.2 (-)
- net IR+: now also C29.1, R25.1, R26.1, U5.5 (+); no longer R32.1
- net IR-: now also C36.1, R31.1, R32.1, U5.6 (-); no longer R27.1, R28.1
- net VL+: now also C28.2, R24.2; no longer C29.1, R24.1, U5.7
- net VL-: now also C27.2, R23.2; no longer C24.1, R19.1, U5.1
- net VR+: now also C34.2, R30.2
- net VR-: now also C31.2, R27.2; no longer R29.1
- net at C23.2, R17.2, R18.2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: now also C25.2, R21.2, R23.1; no longer R20.1
- net at R32.2: now also C36.2, R29.1, R30.1, R31.2, U5.7
- net at C24.2, R19.2, R20.2: now also R22.1, R24.1, U4.7; no longer C25.2, R21.2, U5.2 (-)
- net at C29.2, C32.2, R25.2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: now also R27.1, R28.2, U5.1; no longer R24.2, U5.6 (-)
- new net: C32.1, R28.1, R29.2, U5.2 (-)
- new net: C25.1, R21.1, R22.2, U4.2 (-)
Other:
- note added: "Expected power dissipation: 8-9mA per channel at bipolar zero 12-13mA per channel at full swing"
- note added: "Shown config: High voltage (>9Vpk) low bandwidth (50-65kHz) Alternatives: Low voltage (>4.5Vpk) and/or high bandwith (200-300kHz) HV HB: - Feedback caps 220pF - RC filter caps 3.3nF LV LB: - Feedback resistors 1.5kΩ | 22kΩ - Feedback caps 1.5nF LV HB: - Feedback resistors 1.5kΩ | 22kΩ - Feedback caps 330pF - RC filter caps 3.3nF"
- moved on the sheet: C23, C26, C30, C33, C35, R17, R18, U4A, U4B, U4C

Commit message: HiFiDAC v2 progress
Parts:
- added C39, C42: 10µF 50V, Capacitor_SMD:C_1206_3216Metric, symbol Device:C
- renumbered C23 to C33, C27 to C34, C25 to C35, C28 to C36, C26 to C37, C24 to C38, C30 to C40, C33 to C41, C35 to C43, C29 to C44, C31 to C45, C32 to C46, C34 to C47, C36 to C48, R17 to R15, R18 to R16, R23 to R17, R21 to R18, R22 to R19, R24 to R20, R20 to R21, R19 to R22, R25 to R23, R26 to R24, R27 to R25, R28 to R26, R29 to R27, R30 to R28, R31 to R29, R32 to R30, U4 to U6, U5 to U7
Connections:
- net +15V: now also C39.1, C42.1
- net -15V: now also C39.2, C42.2
- net IL+ renamed I1+
- net IL- renamed I1-
- net IR+ renamed I2+
- net IR- renamed I2-
- net VL+ renamed V1+
- net VL- renamed V1-
- net VR+ renamed V2+
- net VR- renamed V2-
