File: HiFiDAC/i-v-stage.kicad_sch (KiCad schematic)
At the start: 34 parts, among them U6 OPA1612, U7 OPA1612

Commit message: HiFiDAC halved I-V gain
Parts:
- C33, C38, C44, C48: value 1nF C0G -> 1.5nF C0G
- R16, R21, R24, R29: value 3.3kΩRS -> 1.5kΩRS
Other:
- note added: "Shown config: High voltage (>9Vpp) low bandwidth (55-65kHz) Alternatives: Low voltage (>4.5Vpp) and/or high bandwith (250-350kHz) HV HB: - Feedback caps 330pF - RC filter caps 3.3nF LV LB: - Feedback resistors 1.5kΩ | 1.5kΩ - Feedback caps 3.3nF LV HB: - Feedback resistors 1.5kΩ | 1.5kΩ - Feedback caps 470pF - RC filter caps 3.3nF"
- note removed: "Shown config: High voltage (>9Vpk) low bandwidth (50-65kHz) Alternatives: Low voltage (>4.5Vpk) and/or high bandwith (200-300kHz) HV HB: - Feedback caps 220pF - RC filter caps 3.3nF LV LB: - Feedback resistors 1.5kΩ | 22kΩ - Feedback caps 1.5nF LV HB: - Feedback resistors 1.5kΩ | 22kΩ - Feedback caps 330pF - RC filter caps 3.3nF"
Changed lines of the file:
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@@
 		)
 	)
-	(text "Shown config: High voltage (>9Vpk) low bandwidth (50-65kHz)\nAlternatives: Low voltage (>4.5Vpk) and/or high bandwith (200-300kHz)\n\nHV HB:\n - Feedback caps 220pF\n - RC filter caps 3.3nF\nLV LB:\n - Feedback resistors 1.5kΩ | 22kΩ\n - Feedback caps 1.5nF\nLV HB:\n - Feedback resistors 1.5kΩ | 22kΩ\n - Feedback caps 330pF\n - RC filter caps 3.3nF"
+	(text "Shown config: High voltage (>9Vpp) low bandwidth (55-65kHz)\nAlternatives: Low voltage (>4.5Vpp) and/or high bandwith (250-350kHz)\n\nHV HB:\n - Feedback caps 330pF\n - RC filter caps 3.3nF\nLV LB:\n - Feedback resistors 1.5kΩ | 1.5kΩ\n - Feedback caps 3.3nF\nLV HB:\n - Feedback resistors 1.5kΩ | 1.5kΩ\n - Feedback caps 470pF\n - RC filter caps 3.3nF"
 		(exclude_from_sim no)
 		(at 227.33 59.69 0)
@@
 			)
 		)
-		(property "Value" "1nF C0G"
+		(property "Value" "1.5nF C0G"
 			(at 80.01 46.99 90)
 			(effects
@@
 			)
 		)
-		(property "Value" "3.3kΩRS"
+		(property "Value" "1.5kΩRS"
 			(at 80.01 168.91 90)
 			(effects
@@
 			)
 		)
-		(property "Value" "1nF C0G"
+		(property "Value" "1.5nF C0G"
 			(at 80.01 179.07 90)
 			(effects
@@
 			)
 		)
-		(property "Value" "1nF C0G"
+		(property "Value" "1.5nF C0G"
 			(at 80.01 246.38 90)
 			(effects
@@
 			)
 		)
-		(property "Value" "3.3kΩRS"
+		(property "Value" "1.5kΩRS"
 			(at 80.01 127 90)
 			(effects
@@
 			)
 		)
-		(property "Value" "1nF C0G"
+		(property "Value" "1.5nF C0G"
 			(at 80.01 114.3 90)
 			(effects
@@
 			)
 		)
-		(property "Value" "3.3kΩRS"
+		(property "Value" "1.5kΩRS"
 			(at 80.01 36.83 90)
 			(effects
@@
 			)
 		)
-		(property "Value" "3.3kΩRS"
+		(property "Value" "1.5kΩRS"
 			(at 80.01 259.08 90)
 			(effects
