File: CleanLVSupply/CleanLVSupply.kicad_pcb (KiCad board)
At the start: 4 copper layers, 40 x 40 mm, 80 parts, among them J1 12VIN, J2 5V, J3 5V, J4 5V, J5 +-15V, J6 +-15V, U1 LM25576, U2 TPS7A30, U3 LMR64010XMF, U4 TPS7A47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

Commit message: CleanLVSupply build-based updates, v1.1
Parts:
- added CX1: 0.1µF, Capacitor_SMD:C_0603_1608Metric, F.Cu at (151.8, 89.2)
- R4: value 3.09kΩ -> 8.2kΩ
- moved L2 0.44 mm to (154.3, 93.9)
- moved C29 0.12 mm to (153.6, 102.5)
Routing:
- net GND: vias 89 -> 90
Other:
- board text added: "Modular Audio Clean LV Supply v1.1"
- board text removed: "Modular Audio Clean LV Supply"
