File: CleanLVSupply/m15v.kicad_sch (KiCad schematic)
At the start: 31 parts, among them U1 LM25576, U2 TPS7A30

Commit message: CleanLVSupply fixes, HiFiDAC skeleton
Parts:
- R6: value 10kΩ -> 10kΩLN
- R8: value 118kΩ -> 118kΩLN
Changed lines of the file:
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@@
 			)
 		)
-		(property "Value" "10kΩ"
+		(property "Value" "10kΩLN"
 			(at 172.72 129.5399 0)
 			(effects
@@
 			)
 		)
-		(property "Value" "118kΩ"
+		(property "Value" "118kΩLN"
 			(at 172.72 142.2399 0)
 			(effects

Commit message: HiFiDAC routing done, CleanLVSupply fuses added
Connections:
- net -15V_C: no longer R8.2
- new net -15V_SENSE: R8.2
Changed lines of the file:
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@@
-	)
-	(junction
-		(at 170.18 148.59)
-		(diameter 0)
-		(color 0 0 0 0)
 	)
 	(junction
@@
 	(wire
 		(pts
-			(xy 158.75 148.59) (xy 170.18 148.59)
-		)
-		(stroke
-			(width 0)
-			(type default)
-		)
-	)
-	(wire
-		(pts
 			(xy 170.18 69.85) (xy 171.45 69.85)
 		)
@@
 	(wire
 		(pts
-			(xy 170.18 148.59) (xy 170.18 144.78)
-		)
-		(stroke
-			(width 0)
-			(type default)
-		)
-	)
-	(wire
-		(pts
 			(xy 184.15 120.65) (xy 170.18 120.65)
 		)
@@
 	(wire
 		(pts
+			(xy 170.18 144.78) (xy 170.18 156.21)
+		)
+		(stroke
+			(width 0)
+			(type default)
+		)
+	)
+	(wire
+		(pts
 			(xy 217.17 64.77) (xy 195.58 64.77)
 		)
@@
 	(wire
 		(pts
+			(xy 170.18 156.21) (xy 220.98 156.21)
+		)
+		(stroke
+			(width 0)
+			(type default)
+		)
+	)
+	(wire
+		(pts
 			(xy 182.88 73.66) (xy 187.96 73.66)
 		)
@@
 	(wire
 		(pts
-			(xy 184.15 148.59) (xy 170.18 148.59)
+			(xy 158.75 148.59) (xy 184.15 148.59)
 		)
 		(stroke
@@
 		)
 	)
+	(hierarchical_label "-15V_SENSE"
+		(shape input)
+		(at 220.98 156.21 0)
+		(fields_autoplaced yes)
+		(effects
+			(font
+				(size 1.27 1.27)
+			)
+			(justify left)
+		)
+	)

Commit message: CleanLVSupply reduce -17V switch frequency
Parts:
- R4: value 3.09kΩ -> 8.2kΩ
Changed lines of the file:
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@@
 			)
 		)
-		(property "Value" "3.09kΩ"
+		(property "Value" "8.2kΩ"
 			(at 127 80.0099 0)
 			(effects

Commit message: CleanLVSupply build-based updates, v1.1
Parts:
- added CX1: 0.1µF, Capacitor_SMD:C_0603_1608Metric, symbol Device:C
Connections:
- net -17V_SW: now also CX1.2
- net GND: now also CX1.1
Other:
- moved on the sheet: C6, C7
Changed lines of the file:
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@@
 	(paper "A4")
 	(junction
-		(at 231.14 49.53)
-		(diameter 0)
-		(color 0 0 0 0)
-	)
-	(junction
 		(at 201.93 148.59)
 		(diameter 0)
@@
 	)
 	(junction
-		(at 231.14 88.9)
+		(at 231.14 49.53)
 		(diameter 0)
 		(color 0 0 0 0)
@@
 	)
 	(junction
+		(at 231.14 88.9)
+		(diameter 0)
+		(color 0 0 0 0)
+	)
+	(junction
 		(at 110.49 59.69)
 		(diameter 0)
@@
 	)
 	(junction
+		(at 261.62 88.9)
+		(diameter 0)
+		(color 0 0 0 0)
+	)
+	(junction
 		(at 80.01 49.53)
 		(diameter 0)
@@
 	)
 	(junction
-		(at 152.4 128.27)
+		(at 261.62 49.53)
 		(diameter 0)
 		(color 0 0 0 0)
 	)
 	(junction
-		(at 129.54 139.7)
+		(at 152.4 128.27)
 		(diameter 0)
 		(color 0 0 0 0)
 	)
 	(junction
-		(at 247.65 49.53)
+		(at 129.54 139.7)
 		(diameter 0)
 		(color 0 0 0 0)
@@
 	)
 	(junction
-		(at 247.65 88.9)
+		(at 245.11 88.9)
 		(diameter 0)
 		(color 0 0 0 0)
@@
 	)
 	(junction
+		(at 245.11 49.53)
+		(diameter 0)
+		(color 0 0 0 0)
+	)
+	(junction
 		(at 62.23 39.37)
 		(diameter 0)
@@
 	(wire
 		(pts
-			(xy 247.65 88.9) (xy 231.14 88.9)
+			(xy 245.11 88.9) (xy 261.62 88.9)
 		)
 		(stroke
@@
 	(wire
 		(pts
-			(xy 247.65 64.77) (xy 247.65 49.53)
+			(xy 261.62 64.77) (xy 261.62 49.53)
 		)
 		(stroke
@@
 	(wire
 		(pts
+			(xy 261.62 49.53) (xy 266.7 49.53)
+		)
+		(stroke
+			(width 0)
+			(type default)
+		)
+	)
+	(wire
+		(pts
 			(xy 175.26 73.66) (xy 175.26 67.31)
 		)
@@
 	(wire
 		(pts
+			(xy 231.14 49.53) (xy 231.14 64.77)
+		)
+		(stroke
+			(width 0)
+			(type default)
+		)
+	)
+	(wire
+		(pts
+			(xy 231.14 49.53) (xy 245.11 49.53)
+		)
+		(stroke
+			(width 0)
+			(type default)
+		)
+	)
+	(wire
+		(pts
 			(xy 148.59 88.9) (xy 160.02 88.9)
 		)
@@
 	(wire
 		(pts
-			(xy 247.65 49.53) (xy 264.16 49.53)
-		)
-		(stroke
-			(width 0)
-			(type default)
-		)
-	)
-	(wire
-		(pts
 			(xy 138.43 74.93) (xy 138.43 67.31)
 		)
@@
 	(wire
 		(pts
-			(xy 231.14 64.77) (xy 231.14 49.53)
+			(xy 245.11 64.77) (xy 245.11 49.53)
 		)
 		(stroke
@@
 	(wire
 		(pts
-			(xy 231.14 88.9) (xy 217.17 88.9)
+			(xy 217.17 88.9) (xy 231.14 88.9)
 		)
 		(stroke
@@
 	(wire
 		(pts
+			(xy 261.62 88.9) (xy 266.7 88.9)
+		)
+		(stroke
+			(width 0)
+			(type default)
+		)
+	)
+	(wire
+		(pts
 			(xy 101.6 138.43) (xy 101.6 148.59)
 		)
@@
 	(wire
 		(pts
+			(xy 231.14 88.9) (xy 245.11 88.9)
+		)
+		(stroke
+			(width 0)
+			(type default)
+		)
+	)
+	(wire
+		(pts
 			(xy 35.56 39.37) (xy 44.45 39.37)
 		)
@@
 	(wire
 		(pts
-			(xy 231.14 49.53) (xy 217.17 49.53)
+			(xy 217.17 49.53) (xy 231.14 49.53)
 		)
 		(stroke
@@
 	(wire
 		(pts
-			(xy 247.65 88.9) (xy 264.16 88.9)
-		)
-		(stroke
-			(width 0)
-			(type default)
-		)
-	)
-	(wire
-		(pts
 			(xy 182.88 78.74) (xy 175.26 78.74)
 		)
@@
 	(wire
 		(pts
-			(xy 247.65 49.53) (xy 231.14 49.53)
+			(xy 245.11 49.53) (xy 261.62 49.53)
 		)
 		(stroke
@@
 	(wire
 		(pts
-			(xy 247.65 72.39) (xy 247.65 88.9)
+			(xy 261.62 72.39) (xy 261.62 88.9)
 		)
 		(stroke
@@
 	(wire
 		(pts
+			(xy 231.14 72.39) (xy 231.14 88.9)
+		)
+		(stroke
+			(width 0)
+			(type default)
+		)
+	)
+	(wire
+		(pts
 			(xy 67.31 120.65) (xy 83.82 120.65)
 		)
@@
 	(wire
 		(pts
-			(xy 231.14 72.39) (xy 231.14 88.9)
+			(xy 245.11 72.39) (xy 245.11 88.9)
 		)
 		(stroke
@@
 	)
 	(label "-17V_SW"
-		(at 264.16 88.9 0)
+		(at 266.7 88.9 0)
 		(fields_autoplaced yes)
 		(effects
@@
 	(hierarchical_label "GND"
 		(shape input)
-		(at 264.16 49.53 0)
+		(at 266.7 49.53 0)
 		(fields_autoplaced yes)
 		(effects
@@
 	(symbol
 		(lib_id "Device:C_Polarized")
-		(at 247.65 68.58 0)
+		(at 261.62 68.58 0)
 		(unit 1)
 		(exclude_from_sim no)
@@
 		(fields_autoplaced yes)
 		(property "Reference" "C7"
-			(at 251.46 66.4209 0)
+			(at 265.43 66.4209 0)
 			(effects
 				(font
@@
 		)
 		(property "Value" "100µF 25V"
-			(at 251.46 68.9609 0)
+			(at 265.43 68.9609 0)
 			(effects
 				(font
@@
 		)
 		(property "Footprint" "Capacitor_SMD:CP_Elec_6.3x7.7"
-			(at 248.6152 72.39 0)
+			(at 262.5852 72.39 0)
 			(effects
 				(font
@@
 		)
 		(property "Datasheet" "~"
-			(at 247.65 68.58 0)
+			(at 261.62 68.58 0)
 			(effects
 				(font
@@
 		)
 		(property "Description" "Polarized capacitor"
-			(at 247.65 68.58 0)
+			(at 261.62 68.58 0)
 			(effects
 				(font
@@
 	)
 	(symbol
+		(lib_id "Device:C")
+		(at 231.14 68.58 0)
+		(unit 1)
+		(exclude_from_sim no)
+		(in_bom yes)
+		(on_board yes)
+		(dnp no)
+		(fields_autoplaced yes)
+		(property "Reference" "CX1"
+			(at 234.95 67.3099 0)
+			(effects
+				(font
+					(size 1.27 1.27)
+				)
+				(justify left)
+			)
+		)
+		(property "Value" "0.1µF"
+			(at 234.95 69.8499 0)
+			(effects
+				(font
+					(size 1.27 1.27)
+				)
+				(justify left)
+			)
+		)
+		(property "Footprint" "Capacitor_SMD:C_0603_1608Metric"
+			(at 232.1052 72.39 0)
+			(effects
+				(font
+					(size 1.27 1.27)
+				)
+				(hide yes)
+			)
+		)
+		(property "Datasheet" "~"
+			(at 231.14 68.58 0)
+			(effects
+				(font
+					(size 1.27 1.27)
+				)
+				(hide yes)
+			)
+		)
+		(property "Description" "Unpolarized capacitor"
+			(at 231.14 68.58 0)
+			(effects
+				(font
+					(size 1.27 1.27)
+				)
+				(hide yes)
+			)
+		)
+		(pin "2"
+		)
+		(pin "1"
+		)
+		(instances
+			(project "CleanLVSupply"
+				(path "/4327ef59-ef76-48f2-90b1-1a9e4399cfc2/1251894f-ff7f-4119-a254-b437dbce5fd5"
+					(reference "CX1")
+					(unit 1)
+				)
+			)
+		)
+	)
+	(symbol
 		(lib_id "Device:C_Small")
 		(at 180.34 73.66 90)
@@
 	(symbol
 		(lib_id "Device:C")
-		(at 231.14 68.58 0)
+		(at 245.11 68.58 0)
 		(unit 1)
 		(exclude_from_sim no)
@@
 		(fields_autoplaced yes)
 		(property "Reference" "C6"
-			(at 234.95 67.3099 0)
+			(at 248.92 67.3099 0)
 			(effects
 				(font
@@
 		)
 		(property "Value" "1µF 25V"
-			(at 234.95 69.8499 0)
+			(at 248.92 69.8499 0)
 			(effects
 				(font
@@
 		)
 		(property "Footprint" "Capacitor_SMD:C_0603_1608Metric"
-			(at 232.1052 72.39 0)
+			(at 246.0752 72.39 0)
 			(effects
 				(font
@@
 		)
 		(property "Datasheet" "~"
-			(at 231.14 68.58 0)
+			(at 245.11 68.58 0)
 			(effects
 				(font
@@
 		)
 		(property "Description" "Unpolarized capacitor"
-			(at 231.14 68.58 0)
+			(at 245.11 68.58 0)
 			(effects
 				(font
