File: PowerAmplifier/PowerAmplifier.kicad_pcb (KiCad board)
At the start: 4 copper layers, 121 x 40 mm, 156 parts, among them J1 A_SE, J10 AMP, J11 OSC, J12 12V, J13 VADJ, J14 I2C, J15 SWD, J2 AB_IN, J3 AB_BTL, J4 B_SE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

Commit message: PowerAmp+Supply fan LDO change, Supply Rgate fix
Parts:
- U2: value AP2202-ADJ -> TPS7A2401

Commit message: PowerAmpSupply VTRK change
Parts:
- R44: value 24.3kΩ -> 26.1kΩ

Commit message: PowerAmplifier zobel resistor fix
Parts:
- R10, R17, R18, R8: value 1Ω -> 1Ω 0.25W
