File: BluetoothReceiver/BluetoothReceiver.kicad_sch (KiCad schematic)
At the start: 53 parts, among them J1 EXT_ANTENNA, J2 SWD, J3 SPKR/HP, J4 MIC, J5 I2S, J6 I2C/UART, J7 USB, J8 3.3V, U1 STM32F413CHUx

Commit message: BluetoothReceiver PCB mostly done
Parts:
- J3: footprint BW_Connectors:Amphenol_MINITEK_0.8_5P_V -> BW_Connectors:Amphenol_MINITEK_WTB_1.25_5P
- J4: footprint BW_Connectors:Amphenol_MINITEK_0.8_6P_V -> BW_Connectors:Amphenol_MINITEK_WTB_1.25_6P
Connections:
- net PIO3: now also U1.40 (PB4); no longer U1.38 (PA15)
- net PIO5: now also U1.38 (PA15); no longer U1.40 (PB4)
Changed lines of the file:
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@@
 		)
 	)
-	(label "PIO5"
-		(at 55.88 105.41 180)
-		(fields_autoplaced yes)
-		(effects
-			(font
-				(size 1.27 1.27)
-			)
-			(justify right bottom)
-		)
-	)
 	(label "PIO32"
 		(at 55.88 123.19 180)
@@
 	)
 	(label "PIO3"
+		(at 55.88 105.41 180)
+		(fields_autoplaced yes)
+		(effects
+			(font
+				(size 1.27 1.27)
+			)
+			(justify right bottom)
+		)
+	)
+	(label "PIO5"
 		(at 93.98 105.41 0)
 		(fields_autoplaced yes)
@@
 		)
 	)
+	(netclass_flag ""
+		(length 2.54)
+		(shape round)
+		(at 240.03 36.83 180)
+		(fields_autoplaced yes)
+		(effects
+			(font
+				(size 1.27 1.27)
+			)
+			(justify right bottom)
+		)
+		(property "Netclass" "50Ohm"
+			(at 240.7285 39.37 0)
+			(effects
+				(font
+					(size 1.27 1.27)
+					(italic yes)
+				)
+				(justify left)
+			)
+		)
+	)
 	(symbol
 		(lib_id "Device:C_Small")
@@
 			)
 		)
-		(property "Footprint" "BW_Connectors:Amphenol_MINITEK_0.8_6P_V"
+		(property "Footprint" "BW_Connectors:Amphenol_MINITEK_WTB_1.25_6P"
 			(at 275.59 77.47 0)
 			(effects
@@
 			)
 		)
-		(property "Footprint" "BW_Connectors:Amphenol_MINITEK_0.8_5P_V"
+		(property "Footprint" "BW_Connectors:Amphenol_MINITEK_WTB_1.25_5P"
 			(at 242.57 64.77 0)
 			(effects
