File: BlockBoxController/BlockBoxController.kicad_sch (KiCad schematic)
At the start: 33 parts, among them J1 SWD, J2 3.3V, U1 STM32H725VGTx

Commit message: BlockBoxController schematic done for now
Parts:
- removed J2: 3.3V, BW_Connectors:Amphenol_MINITEK_WTB_1.25_2P, symbol Connector:Conn_01x02_Pin
- added C27: 220µF 16V, Capacitor_SMD:CP_Elec_6.3x7.7, symbol Device:C_Polarized
- added C28: 220µF 6.3V, Capacitor_SMD:CP_Elec_5x5.8, symbol Device:C_Polarized
- added J1: B1_SWLED, Connector_PinHeader_2.54mm:PinHeader_1x03_P2.54mm_Vertical, symbol Connector:Conn_01x03_Pin
- added J10: I2C1/USART1, BW_Connectors:Amphenol_MINITEK_WTB_1.25_4P, symbol Connector:Conn_01x04_Pin
- added J11: I2C4/UART4, BW_Connectors:Amphenol_MINITEK_WTB_1.25_3P, symbol Connector:Conn_01x03_Pin
- added J12: B1_LED_BRIGHTNESS, Connector_PinHeader_2.54mm:PinHeader_1x03_P2.54mm_Vertical, symbol Connector:Conn_01x03_Pin
- added J13: I2C5, BW_Connectors:PinHeader_3x05_P2.54mm_Vertical, symbol Connector:Conn_01x15_Pin
- added J14: B1_BTN, Connector_PinHeader_2.54mm:PinHeader_2x06_P2.54mm_Vertical, symbol Connector_Generic:Conn_02x06_Odd_Even
- added J15: PWR, Connector_Molex:Molex_Nano-Fit_105309-xx04_1x04_P2.50mm_Vertical, symbol Connector:Conn_01x04_Pin
- added J3: NHD-3.5-320240FT-CON, BW_Connectors:PinHeader_2x09_P2.54mm_Vertical_Mirrored, symbol BW_Active:NHD-3.5-320240FT-CON
- added J4: CHG, BW_Connectors:Amphenol_MINITEK_WTB_1.25_5P, symbol Connector:Conn_01x05_Pin
- added J5: AMP, BW_Connectors:Amphenol_MINITEK_WTB_1.25_4P, symbol Connector:Conn_01x04_Pin
- added J6: I2S, BW_Connectors:Amphenol_MINITEK_WTB_1.25_4P, symbol Connector:Conn_01x04_Pin
- added J7: B1_LCD_SWITCH, Connector_PinHeader_2.54mm:PinHeader_1x02_P2.54mm_Vertical, symbol Connector:Conn_01x02_Pin
- added J8: LED, Connector_PinHeader_2.54mm:PinHeader_1x04_P2.54mm_Vertical, symbol Connector:Conn_01x04_Pin
- added J9: B1_LEDMODE, Connector_PinHeader_2.54mm:PinHeader_1x03_P2.54mm_Vertical, symbol Connector:Conn_01x03_Pin
- added JP1: VBL, Jumper:SolderJumper-3_P1.3mm_Open_RoundedPad1.0x1.5mm, symbol Jumper:SolderJumper_3_Open
- added Q1, Q2: NX138BK, Package_TO_SOT_SMD:SOT-23, symbol Device:Q_NMOS_GSD
- added Q3, Q4, Q5, Q6: DMG2302UK, Package_TO_SOT_SMD:SOT-23, symbol Device:Q_NMOS_GSD
- added R1, R2, R3, R4, R6, R7: 50/100Ω, Resistor_SMD:R_0603_1608Metric, symbol Device:R_US
- added R11: 10Ω, Resistor_SMD:R_0603_1608Metric, symbol Device:R_US
- added R12, R13: 27Ω, Resistor_SMD:R_0603_1608Metric, symbol Device:R_US
- added R14, R15, R16, R17, R8, R9: 4.7kΩ, Resistor_SMD:R_0603_1608Metric, symbol Device:R_US
- added R18, R19, R20, R21: 0Ω, Resistor_SMD:R_0603_1608Metric, symbol Device:R_US
- added R22, R23: 1kΩ, Resistor_SMD:R_0603_1608Metric, symbol Device:R_US
- added RV1: 35WR10K, BW_PassiveMechanical:Potentiometer_TT_35W, symbol Device:R_Potentiometer_Trim_US
- added TP1: DEBUG_TX, BW_PassiveMechanical:TP_0603_1608Metric_Fused, symbol Connector:TestPoint_Small
- added TP10: I2C1_SCL/USART1_TX, BW_PassiveMechanical:TP_0603_1608Metric_Fused, symbol Connector:TestPoint_Small
- added TP11: I2C1_SDA/USART1_RX, BW_PassiveMechanical:TP_0603_1608Metric_Fused, symbol Connector:TestPoint_Small
- added TP12: I2C4_SCL/UART4_RX, BW_PassiveMechanical:TP_0603_1608Metric_Fused, symbol Connector:TestPoint_Small
- added TP13: I2C4_SDA/UART4_TX, BW_PassiveMechanical:TP_0603_1608Metric_Fused, symbol Connector:TestPoint_Small
- added TP14: I2C5_SDA, BW_PassiveMechanical:TP_0603_1608Metric_Fused, symbol Connector:TestPoint_Small
- added TP15: I2C5_SCL, BW_PassiveMechanical:TP_0603_1608Metric_Fused, symbol Connector:TestPoint_Small
- added TP2: DEBUG_RX, BW_PassiveMechanical:TP_0603_1608Metric_Fused, symbol Connector:TestPoint_Small
- added TP3: CHG_SMB_SCL, BW_PassiveMechanical:TP_0603_1608Metric_Fused, symbol Connector:TestPoint_Small
- added TP4: CHG_SMB_SDA, BW_PassiveMechanical:TP_0603_1608Metric_Fused, symbol Connector:TestPoint_Small
- added TP5: CHG_ACOK, BW_PassiveMechanical:TP_0603_1608Metric_Fused, symbol Connector:TestPoint_Small
- added TP6: AMP_~{CLIP_OTW}, TestPoint:TestPoint_Pad_D1.0mm, symbol Connector:TestPoint_Small
- added TP7: CHG_IOUT, TestPoint:TestPoint_Pad_D1.0mm, symbol Connector:TestPoint_Small
- added TP8: AMP_~{FAULT}, TestPoint:TestPoint_Pad_D1.0mm, symbol Connector:TestPoint_Small
- added TP9: AMP_~{RESET}, TestPoint:TestPoint_Pad_D1.0mm, symbol Connector:TestPoint_Small
- renumbered C7 to C10, C8 to C11, C9 to C12, C10 to C13, C22 to C14, C25 to C15, C5 to C16, C12 to C17, C13 to C18, C18 to C19, C19 to C20, C20 to C21, C27 to C22, C26 to C23, C14 to C24, C15 to C25, C16 to C26, C17 to C29, C21 to C5, C23 to C6, C24 to C7, C11 to C8, C6 to C9, J1 to J2, R2 to R10, R1 to R5
Connections:
- net +3.3V: now also J12.1 (Pin_1), J15.3 (Pin_3), J3.2 (VDD), JP1.1 (A), R14.1, R15.1, R16.1, R17.1, R22.1, R23.1, R8.1, R9.1, RV1.3
- net AMP_~{CLIP_OTW}: now also J5.3 (Pin_3), TP6.1
- net AMP_~{FAULT}: now also J5.2 (Pin_2), TP8.1
- net AMP_~{RESET}: now also J5.1 (Pin_1), TP9.1
- net B1_BACK: now also J14.6 (Pin_6)
- net B1_FWD: now also J14.12 (Pin_12)
- net B1_LCD_SWITCH: now also J7.1 (Pin_1)
- net B1_LEDMODE_1: now also J9.1 (Pin_1)
- net B1_LEDMODE_2: now also J9.3 (Pin_3)
- net B1_LED_BRIGHTNESS: now also J12.2 (Pin_2)
- net B1_MFB: now also J14.10 (Pin_10)
- net B1_PLAY: now also J14.8 (Pin_8)
- net B1_SWLED_MAIN: now also Q1.1 (G)
- net B1_SWLED_PWR: now also Q2.1 (G)
- net B1_VOL_DOWN: now also J14.4 (Pin_4)
- net B1_VOL_UP: now also J14.2 (Pin_2)
- net CHG_ACOK: now also J4.3 (Pin_3), TP5.1
- net CHG_IOUT: now also J4.4 (Pin_4), TP7.1
- net CHG_SMB_SCL: now also J4.1 (Pin_1), R8.2, TP3.1
- net CHG_SMB_SDA: now also J4.2 (Pin_2), R9.2, TP4.1
- net DEBUG_RX: now also TP2.1
- net DEBUG_TX: now also TP1.1
- net GND: now also C27.2, C28.2, J10.4 (Pin_4), J11.3 (Pin_3), J12.3 (Pin_3), J14.1 (Pin_1), J14.11 (Pin_11), J14.3 (Pin_3), J14.5 (Pin_5), J14.7 (Pin_7), J14.9 (Pin_9), J15.4 (Pin_4), J3.1 (GND), J4.5 (Pin_5), J5.4 (Pin_4), J6.4 (Pin_4), J7.2 (Pin_2), J9.2 (Pin_2), Q1.2 (S), Q2.2 (S), Q3.2 (S), Q4.2 (S), Q5.2 (S), Q6.2 (S), RV1.1
- net I2C1_SCL/USART1_TX: now also J10.1 (Pin_1), R14.2, TP10.1
- net I2C1_SDA/USART1_RX: now also J10.2 (Pin_2), R15.2, TP11.1
- net I2C1_~{INT0}: now also J10.3 (Pin_3)
- net I2C4_SCL/UART4_RX: now also J11.1 (Pin_1), R16.2, TP12.1
- net I2C4_SDA/UART4_TX: now also J11.2 (Pin_2), R17.2, TP13.1
- net I2C5_SCL: now also J13.1 (Pin_1), J13.10 (Pin_10), J13.13 (Pin_13), J13.4 (Pin_4), J13.7 (Pin_7), R22.2, TP15.1
- net I2C5_SDA: now also J13.11 (Pin_11), J13.14 (Pin_14), J13.2 (Pin_2), J13.5 (Pin_5), J13.8 (Pin_8), R23.2, TP14.1
- net I2C5_~{INT0}: now also J13.3 (Pin_3)
- net I2C5_~{INT1}: now also J13.6 (Pin_6)
- net I2C5_~{INT2}: now also J13.9 (Pin_9)
- net I2C5_~{INT3}: now also J13.12 (Pin_12)
- net I2C5_~{INT4}: now also J13.15 (Pin_15)
- net I2S_BCK: now also R11.1
- net I2S_DATA: now also R12.1
- net I2S_LRCK: now also R13.1
- net LCD_ALT_MISO: now also R20.1
- net LCD_ALT_MOSI: now also R21.1
- net LCD_ALT_SCK: now also R19.1
- net LCD_ALT_~{CS}: now also R18.1
- net LCD_B1_D3: now also J3.10 (AUDIO_L)
- net LCD_BL_DRV: now also Q3.1 (G)
- net LCD_GPIO2/B1_D6: now also J3.13 (GPIO2)
- net LCD_GPIO3/B1_D7: now also J3.14 (GPIO3)
- net LCD_IO0/MOSI/B1_~{E}: now also R21.2, R4.2
- net LCD_IO1/MISO/B1_RW: now also R1.1, R20.2
- net LCD_IO2/GPIO0/B1_D4: now also R7.2
- net LCD_IO3/GPIO1/B1_D5: now also R6.1
- net LCD_SCK/B1_RS: now also R19.2, R2.2
- net LCD_~{CS}/B1_D0: now also R18.2, R3.1
- net LCD_~{INT}/B1_D1: now also J3.8 (~{INT})
- net LCD_~{PD}/B1_D2: now also J3.9 (~{PD})
- net LED_B: now also Q6.1 (G)
- net LED_G: now also Q5.1 (G)
- net LED_R: now also Q4.1 (G)
- new net: J6.1 (Pin_1), R11.2
- new net: J6.2 (Pin_2), R12.2
- new net: J6.3 (Pin_3), R13.2
- new net: J1.2 (Pin_2), Q1.3 (D)
- new net: J3.15 (VBL), J3.17 (VBL), JP1.2 (C)
- new net: J3.6 (MOSI/IO0), R4.1
- new net: J8.3 (Pin_3), Q4.3 (D)
- new net: J8.2 (Pin_2), Q5.3 (D)
- new net: J8.4 (Pin_4), Q6.3 (D)
- new net: J3.5 (MISO/IO1), R1.2
- new net: J3.12 (GPIO1/IO3), R6.2
- new net: J3.16 (GND_BL), J3.18 (GND_BL), Q3.3 (D)
- new net: J1.3 (Pin_3), Q2.3 (D)
- new net: J3.11 (GPIO0/IO2), R7.1
- new net: J3.3 (NC1), RV1.2
- new net: J3.4 (SCK), R2.1
- new net: J3.7 (~{CS}), R3.2
- new net +12V: C27.1, J15.1 (Pin_1), J8.1 (Pin_1)
- new net +5V: C28.1, J1.1 (Pin_1), J15.2 (Pin_2), JP1.3 (B)
Other:
- note added: "3x5-pin connector Rows: SCL, SDA, INT0-4"
- note added: "Can replace with shunt for BlockBox v2"
- note added: "Choose termination resistors based on cable for BlockBox v2 (flat cable ≈100Ω, Cat7 ≈50Ω) Terminate IO0-IO3 equally on LCD side!"
- note added: "Populate for BlockBox v1 (contrast)"
- note added: "Remove resistors for UART"
- note added: "Remove resistors for USART"
- moved on the sheet: C1, C10, C11, C12, C13, C14, C15, C16, C17, C18, C19, C2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
