File: BatteryMonitor/BatteryMonitor.kicad_pcb (KiCad board)
At the start: 4 copper layers, 40 x 40 mm, 71 parts, among them J1 SWD, J2 BAT+, J3 BAL_THERM, J4 I2C, J5 BAT-, J6 PACK_OUT, J7 PWR_SWITCH, Q1 NX138BK, Q2 NTMFS0D6N04XM, Q3 NTMFS0D6N04XM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

Commit message: BatteryMonitor doubled FET protection zener
Single zener causes excessive leakage when off; opposite-polarity pair fixes that
Parts:
- added D3: BZT52C15, Diode_SMD:D_SOD-123, F.Cu at (161.1, 110.3)
- moved D2 3.57 mm to (157.5, 109.1), turned to 90 degrees
- renumbered D3 to D4
Connections:
- C24 pad 2: Net-(D2-A) -> Net-(D3-K)
- C25 pad 2: Net-(D2-A) -> Net-(D3-K)
- J6 pad 1: Net-(D2-A) -> Net-(D3-K)
- Q3 pad 1: Net-(D2-A) -> Net-(D3-K)
- R19 pad 2: Net-(D2-A) -> Net-(D3-K)
Routing:
- net Net-(D3-K): track 0.00 -> 32.4 mm
- net Net-(D2-A): track 32.6 -> 3.55 mm
- net Net-(D2-K): track 8.69 -> 7.55 mm
Other:
- board text added: "Modular Audio Battery Monitor v1.2"
- board text removed: "Modular Audio Battery Monitor v1.1"
