File: BasePower/12v-buck-boost.kicad_sch (KiCad schematic)
At the start: 24 parts, among them U1 TPS552892

Commit message: BasePower design and inventory done
Parts:
- added C2, C3: ?pF, Capacitor_SMD:C_0603_1608Metric, symbol Device:C_Small
- added R4, R5: ?Ω, Resistor_SMD:R_1206_3216Metric, symbol Device:R_US
- added R6, R7: 50Ω, Resistor_SMD:R_0603_1608Metric, symbol Device:R_Small_US
- added TP1: SW1, Connector_Coaxial:U.FL_Molex_MCRF_73412-0110_Vertical, symbol Connector:Conn_Coaxial_Small
- added TP2: SW2, Connector_Coaxial:U.FL_Molex_MCRF_73412-0110_Vertical, symbol Connector:Conn_Coaxial_Small
- renumbered C8 to C10, C9 to C11, C10 to C12, C11 to C13, C12 to C14, C13 to C15, C14 to C16, C15 to C17, C16 to C18, C2 to C4, C3 to C5, C4 to C6, C5 to C7, C6 to C8, C7 to C9, R6 to R10, R7 to R11, R8 to R12, R9 to R13, R10 to R14, R4 to R8, R5 to R9
Connections:
- net GND: now also R4.1, R5.1, TP1.2 (Ext), TP2.2 (Ext)
- net at C5.1, L1.2, U1.10 (SW2): now also C3.2, R7.1
- net at C4.1, L1.1, U1.8 (SW1): now also C2.2, R6.1
- new net: R7.2, TP2.1 (In)
- new net: R6.2, TP1.1 (In)
- new net: C3.1, R5.2
- new net: C2.1, R4.2
Other:
- note removed: "Test points and snubber footprints? Depending on board space"

Commit message: BasePower v1.2 + inventory
Added 12V clean LDO and improved power good display
Parts:
- removed R10: 10kΩ, Resistor_SMD:R_0603_1608Metric, symbol Device:R_US
- renumbered R4 to R10, R5 to R11, R6 to R12, R7 to R13, R8 to R14, R9 to R15, R11 to R16, R12 to R17, R13 to R18, R14 to R19
Other:
- note added: "Add large resistor (≈1MΩ) in parallel for slightly higher output"
Changed lines of the file:
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@@
 	)
 	(junction
-		(at 105.41 102.87)
-		(diameter 0)
-		(color 0 0 0 0)
-	)
-	(junction
 		(at 138.43 133.35)
 		(diameter 0)
@@
 	(wire
 		(pts
-			(xy 107.95 105.41) (xy 105.41 105.41)
-		)
-		(stroke
-			(width 0)
-			(type default)
-		)
-	)
-	(wire
-		(pts
 			(xy 140.97 128.27) (xy 166.37 128.27)
 		)
@@
 	(wire
 		(pts
-			(xy 101.6 102.87) (xy 105.41 102.87)
-		)
-		(stroke
-			(width 0)
-			(type default)
-		)
-	)
-	(wire
-		(pts
 			(xy 80.01 95.25) (xy 80.01 133.35)
 		)
@@
 	(wire
 		(pts
-			(xy 93.98 102.87) (xy 88.9 102.87)
-		)
-		(stroke
-			(width 0)
-			(type default)
-		)
-	)
-	(wire
-		(pts
 			(xy 88.9 123.19) (xy 88.9 128.27)
 		)
@@
 	(wire
 		(pts
-			(xy 88.9 102.87) (xy 88.9 113.03)
-		)
-		(stroke
-			(width 0)
-			(type default)
-		)
-	)
-	(wire
-		(pts
 			(xy 198.12 113.03) (xy 198.12 114.3)
 		)
@@
 	(wire
 		(pts
-			(xy 105.41 102.87) (xy 119.38 102.87)
+			(xy 114.3 102.87) (xy 119.38 102.87)
 		)
 		(stroke
@@
 	(wire
 		(pts
-			(xy 105.41 105.41) (xy 105.41 102.87)
-		)
-		(stroke
-			(width 0)
-			(type default)
-		)
-	)
-	(wire
-		(pts
 			(xy 149.86 82.55) (xy 149.86 85.09)
 		)
@@
 		)
 	)
+	(text "Add large resistor (≈1MΩ)\nin parallel for\nslightly higher output"
+		(exclude_from_sim no)
+		(at 265.43 117.856 0)
+		(effects
+			(font
+				(size 1.27 1.27)
+			)
+		)
+	)
 	(text "Ideal AGND-PGND\nconnection point"
 		(exclude_from_sim no)
@@
 	(hierarchical_label "PG"
 		(shape output)
-		(at 107.95 105.41 0)
+		(at 114.3 102.87 180)
 		(fields_autoplaced yes)
 		(effects
@@
 				(size 1.27 1.27)
 			)
-			(justify left)
+			(justify right)
 		)
 	)
@@
 		(dnp no)
 		(fields_autoplaced yes)
-		(property "Reference" "#PWR011"
+		(property "Reference" "#PWR012"
 			(at 138.43 140.97 0)
 			(effects
@@
 			(project ""
 				(path "/7a4c470e-f21a-4fdb-85db-575cfe7b758f/bd3e5906-e3f2-44b3-9d24-6c6002848911"
-					(reference "#PWR011")
+					(reference "#PWR012")
 					(unit 1)
 				)
@@
 		(dnp no)
 		(fields_autoplaced yes)
-		(property "Reference" "#PWR08"
+		(property "Reference" "#PWR09"
 			(at 139.7 62.23 0)
 			(effects
@@
 			(project "BasePower"
 				(path "/7a4c470e-f21a-4fdb-85db-575cfe7b758f/bd3e5906-e3f2-44b3-9d24-6c6002848911"
-					(reference "#PWR08")
+					(reference "#PWR09")
 					(unit 1)
 				)
@@
 		(dnp no)
 		(fields_autoplaced yes)
-		(property "Reference" "R7"
+		(property "Reference" "R13"
 			(at 163.83 68.58 90)
 			(effects
@@
 			(project "BasePower"
 				(path "/7a4c470e-f21a-4fdb-85db-575cfe7b758f/bd3e5906-e3f2-44b3-9d24-6c6002848911"
-					(reference "R7")
+					(reference "R13")
 					(unit 1)
 				)
@@
 		(dnp no)
 		(fields_autoplaced yes)
-		(property "Reference" "R11"
+		(property "Reference" "R16"
 			(at 200.66 115.5699 0)
 			(effects
@@
 			(project "BasePower"
 				(path "/7a4c470e-f21a-4fdb-85db-575cfe7b758f/bd3e5906-e3f2-44b3-9d24-6c6002848911"
-					(reference "R11")
+					(reference "R16")
 					(unit 1)
 				)
@@
 		(dnp no)
 		(fields_autoplaced yes)
-		(property "Reference" "#PWR010"
+		(property "Reference" "#PWR011"
 			(at 181.61 74.93 0)
 			(effects
@@
 			(project "BasePower"
 				(path "/7a4c470e-f21a-4fdb-85db-575cfe7b758f/bd3e5906-e3f2-44b3-9d24-6c6002848911"
-					(reference "#PWR010")
+					(reference "#PWR011")
 					(unit 1)
 				)
@@
 		(dnp no)
 		(fields_autoplaced yes)
-		(property "Reference" "R6"
+		(property "Reference" "R12"
 			(at 115.57 68.58 90)
 			(effects
@@
 			(project "BasePower"
 				(path "/7a4c470e-f21a-4fdb-85db-575cfe7b758f/bd3e5906-e3f2-44b3-9d24-6c6002848911"
-					(reference "R6")
+					(reference "R12")
 					(unit 1)
 				)
@@
 		(dnp yes)
 		(fields_autoplaced yes)
-		(property "Reference" "R4"
+		(property "Reference" "R10"
 			(at 127 59.6899 0)
 			(effects
@@
 			(project "BasePower"
 				(path "/7a4c470e-f21a-4fdb-85db-575cfe7b758f/bd3e5906-e3f2-44b3-9d24-6c6002848911"
-					(reference "R4")
+					(reference "R10")
 					(unit 1)
 				)
@@
 	)
 	(symbol
-		(lib_id "Device:R_US")
-		(at 97.79 102.87 90)
-		(unit 1)
-		(exclude_from_sim no)
-		(in_bom yes)
-		(on_board yes)
-		(dnp no)
-		(fields_autoplaced yes)
-		(property "Reference" "R10"
-			(at 97.79 106.68 90)
-			(effects
-				(font
-					(size 1.27 1.27)
-				)
-			)
-		)
-		(property "Value" "10kΩ"
-			(at 97.79 109.22 90)
-			(effects
-				(font
-					(size 1.27 1.27)
-				)
-			)
-		)
-		(property "Footprint" "Resistor_SMD:R_0603_1608Metric"
-			(at 98.044 101.854 90)
-			(effects
-				(font
-					(size 1.27 1.27)
-				)
-				(hide yes)
-			)
-		)
-		(property "Datasheet" "~"
-			(at 97.79 102.87 0)
-			(effects
-				(font
-					(size 1.27 1.27)
-				)
-				(hide yes)
-			)
-		)
-		(property "Description" "Resistor, US symbol"
-			(at 97.79 102.87 0)
-			(effects
-				(font
-					(size 1.27 1.27)
-				)
-				(hide yes)
-			)
-		)
-		(pin "1"
-		)
-		(pin "2"
-		)
-		(instances
-			(project "BasePower"
-				(path "/7a4c470e-f21a-4fdb-85db-575cfe7b758f/bd3e5906-e3f2-44b3-9d24-6c6002848911"
-					(reference "R10")
-					(unit 1)
-				)
-			)
-		)
-	)
-	(symbol
 		(lib_id "Device:C_Small")
 		(at 69.85 113.03 0)
@@
 		(dnp yes)
 		(fields_autoplaced yes)
-		(property "Reference" "R5"
+		(property "Reference" "R11"
 			(at 152.4 59.6899 0)
 			(effects
@@
 			(project "BasePower"
 				(path "/7a4c470e-f21a-4fdb-85db-575cfe7b758f/bd3e5906-e3f2-44b3-9d24-6c6002848911"
-					(reference "R5")
+					(reference "R11")
 					(unit 1)
 				)
@@
 		(on_board yes)
 		(dnp no)
-		(property "Reference" "R12"
+		(property "Reference" "R17"
 			(at 246.38 116.8399 0)
 			(effects
@@
 			(project "BasePower"
 				(path "/7a4c470e-f21a-4fdb-85db-575cfe7b758f/bd3e5906-e3f2-44b3-9d24-6c6002848911"
-					(reference "R12")
+					(reference "R17")
 					(unit 1)
 				)
@@
 		(dnp no)
 		(fields_autoplaced yes)
-		(property "Reference" "#PWR09"
+		(property "Reference" "#PWR010"
 			(at 97.79 74.93 0)
 			(effects
@@
 			(project "BasePower"
 				(path "/7a4c470e-f21a-4fdb-85db-575cfe7b758f/bd3e5906-e3f2-44b3-9d24-6c6002848911"
-					(reference "#PWR09")
+					(reference "#PWR010")
 					(unit 1)
 				)
@@
 		(dnp no)
 		(fields_autoplaced yes)
-		(property "Reference" "R13"
+		(property "Reference" "R18"
 			(at 111.76 123.1899 0)
 			(effects
@@
 			(project ""
 				(path "/7a4c470e-f21a-4fdb-85db-575cfe7b758f/bd3e5906-e3f2-44b3-9d24-6c6002848911"
-					(reference "R13")
+					(reference "R18")
 					(unit 1)
 				)
@@
 		(dnp no)
 		(fields_autoplaced yes)
-		(property "Reference" "R9"
+		(property "Reference" "R15"
 			(at 246.38 95.2499 0)
 			(effects
@@
 			(project "BasePower"
 				(path "/7a4c470e-f21a-4fdb-85db-575cfe7b758f/bd3e5906-e3f2-44b3-9d24-6c6002848911"
-					(reference "R9")
+					(reference "R15")
 					(unit 1)
 				)
@@
 		(dnp yes)
 		(fields_autoplaced yes)
-		(property "Reference" "R14"
+		(property "Reference" "R19"
 			(at 168.91 123.1899 0)
 			(effects
@@
 			(project "BasePower"
 				(path "/7a4c470e-f21a-4fdb-85db-575cfe7b758f/bd3e5906-e3f2-44b3-9d24-6c6002848911"
-					(reference "R14")
+					(reference "R19")
 					(unit 1)
 				)
@@
 		(dnp no)
 		(fields_autoplaced yes)
-		(property "Reference" "R8"
+		(property "Reference" "R14"
 			(at 234.95 78.74 90)
 			(effects
@@
 			(project "BasePower"
 				(path "/7a4c470e-f21a-4fdb-85db-575cfe7b758f/bd3e5906-e3f2-44b3-9d24-6c6002848911"
-					(reference "R8")
+					(reference "R14")
 					(unit 1)
 				)
