File: BasePower/3.3v-buck.kicad_sch (KiCad schematic)
At the start: 12 parts, among them U3 TPSM33625F

Commit message: BasePower design and inventory done
Parts:
- renumbered C25 to C27, C26 to C28, C27 to C29, C28 to C30, C29 to C31, C30 to C32, R16 to R20, R17 to R21, R18 to R22, R19 to R23, R20 to R24
Changed lines of the file:
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@@
 		(dnp no)
 		(fields_autoplaced yes)
-		(property "Reference" "C29"
+		(property "Reference" "C31"
 			(at 106.68 100.3362 0)
 			(effects
@@
 			(project "BasePower"
 				(path "/7a4c470e-f21a-4fdb-85db-575cfe7b758f/66a6072f-b93c-48b6-9ad2-cc693c587a24"
-					(reference "C29")
+					(reference "C31")
 					(unit 1)
 				)
@@
 		(dnp no)
 		(fields_autoplaced yes)
-		(property "Reference" "C30"
+		(property "Reference" "C32"
 			(at 118.11 100.3362 0)
 			(effects
@@
 			(project "BasePower"
 				(path "/7a4c470e-f21a-4fdb-85db-575cfe7b758f/66a6072f-b93c-48b6-9ad2-cc693c587a24"
-					(reference "C30")
+					(reference "C32")
 					(unit 1)
 				)
@@
 		(dnp no)
 		(fields_autoplaced yes)
-		(property "Reference" "R16"
+		(property "Reference" "R20"
 			(at 95.25 85.0899 0)
 			(effects
@@
 			(project "BasePower"
 				(path "/7a4c470e-f21a-4fdb-85db-575cfe7b758f/66a6072f-b93c-48b6-9ad2-cc693c587a24"
-					(reference "R16")
+					(reference "R20")
 					(unit 1)
 				)
@@
 		(on_board yes)
 		(dnp no)
-		(property "Reference" "C26"
+		(property "Reference" "C28"
 			(at 203.2 90.1762 0)
 			(effects
@@
 			(project "BasePower"
 				(path "/7a4c470e-f21a-4fdb-85db-575cfe7b758f/66a6072f-b93c-48b6-9ad2-cc693c587a24"
-					(reference "C26")
+					(reference "C28")
 					(unit 1)
 				)
@@
 		(dnp no)
 		(fields_autoplaced yes)
-		(property "Reference" "C27"
+		(property "Reference" "C29"
 			(at 224.79 89.2809 0)
 			(effects
@@
 			(project "BasePower"
 				(path "/7a4c470e-f21a-4fdb-85db-575cfe7b758f/66a6072f-b93c-48b6-9ad2-cc693c587a24"
-					(reference "C27")
+					(reference "C29")
 					(unit 1)
 				)
@@
 		(dnp no)
 		(fields_autoplaced yes)
-		(property "Reference" "#PWR08"
+		(property "Reference" "#PWR013"
 			(at 128.27 118.11 0)
 			(effects
@@
 			(project "BasePower"
 				(path "/7a4c470e-f21a-4fdb-85db-575cfe7b758f/66a6072f-b93c-48b6-9ad2-cc693c587a24"
-					(reference "#PWR08")
+					(reference "#PWR013")
 					(unit 1)
 				)
@@
 		(dnp no)
 		(fields_autoplaced yes)
-		(property "Reference" "C25"
+		(property "Reference" "C27"
 			(at 121.92 85.0962 0)
 			(effects
@@
 			(project "BasePower"
 				(path "/7a4c470e-f21a-4fdb-85db-575cfe7b758f/66a6072f-b93c-48b6-9ad2-cc693c587a24"
-					(reference "C25")
+					(reference "C27")
 					(unit 1)
 				)
@@
 		(dnp no)
 		(fields_autoplaced yes)
-		(property "Reference" "R17"
+		(property "Reference" "R21"
 			(at 173.99 90.1699 0)
 			(effects
@@
 			(project "BasePower"
 				(path "/7a4c470e-f21a-4fdb-85db-575cfe7b758f/66a6072f-b93c-48b6-9ad2-cc693c587a24"
-					(reference "R17")
+					(reference "R21")
 					(unit 1)
 				)
@@
 		(dnp no)
 		(fields_autoplaced yes)
-		(property "Reference" "C28"
+		(property "Reference" "C30"
 			(at 80.01 93.9862 0)
 			(effects
@@
 			(project "BasePower"
 				(path "/7a4c470e-f21a-4fdb-85db-575cfe7b758f/66a6072f-b93c-48b6-9ad2-cc693c587a24"
-					(reference "C28")
+					(reference "C30")
 					(unit 1)
 				)
@@
 		(on_board yes)
 		(dnp no)
-		(property "Reference" "R19"
+		(property "Reference" "R23"
 			(at 95.25 100.3299 0)
 			(effects
@@
 			(project "BasePower"
 				(path "/7a4c470e-f21a-4fdb-85db-575cfe7b758f/66a6072f-b93c-48b6-9ad2-cc693c587a24"
-					(reference "R19")
+					(reference "R23")
 					(unit 1)
 				)
@@
 		(dnp no)
 		(fields_autoplaced yes)
-		(property "Reference" "R18"
+		(property "Reference" "R22"
 			(at 186.69 90.1699 0)
 			(effects
@@
 			(project "BasePower"
 				(path "/7a4c470e-f21a-4fdb-85db-575cfe7b758f/66a6072f-b93c-48b6-9ad2-cc693c587a24"
-					(reference "R18")
+					(reference "R22")
 					(unit 1)
 				)
@@
 		(on_board yes)
 		(dnp no)
-		(property "Reference" "R20"
+		(property "Reference" "R24"
 			(at 186.69 102.8699 0)
 			(effects
@@
 			(project "BasePower"
 				(path "/7a4c470e-f21a-4fdb-85db-575cfe7b758f/66a6072f-b93c-48b6-9ad2-cc693c587a24"
-					(reference "R20")
-					(unit 1)
-				)
+					(reference "R24")
+					(unit 1)
+				)

Commit message: BasePower v1.2 + inventory
Added 12V clean LDO and improved power good display
Parts:
- removed R21: 10kΩ, Resistor_SMD:R_0603_1608Metric, symbol Device:R_US
- renumbered R20 to R24, R22 to R25, R23 to R26, R24 to R27
Changed lines of the file:
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@@
-	)
-	(junction
-		(at 171.45 100.33)
-		(diameter 0)
-		(color 0 0 0 0)
 	)
 	(junction
@@
 	(junction
 		(at 184.15 110.49)
-		(diameter 0)
-		(color 0 0 0 0)
-	)
-	(junction
-		(at 171.45 85.09)
 		(diameter 0)
 		(color 0 0 0 0)
@@
 	(wire
 		(pts
-			(xy 171.45 95.25) (xy 171.45 100.33)
-		)
-		(stroke
-			(width 0)
-			(type default)
-		)
-	)
-	(wire
-		(pts
 			(xy 68.58 80.01) (xy 77.47 80.01)
 		)
@@
 	(wire
 		(pts
-			(xy 171.45 85.09) (xy 184.15 85.09)
+			(xy 163.83 85.09) (xy 184.15 85.09)
 		)
 		(stroke
@@
 	(wire
 		(pts
-			(xy 171.45 85.09) (xy 171.45 87.63)
-		)
-		(stroke
-			(width 0)
-			(type default)
-		)
-	)
-	(wire
-		(pts
 			(xy 161.29 90.17) (xy 163.83 90.17)
 		)
@@
 	(wire
 		(pts
-			(xy 171.45 100.33) (xy 161.29 100.33)
+			(xy 161.29 100.33) (xy 163.83 100.33)
 		)
 		(stroke
@@
 	(wire
 		(pts
-			(xy 171.45 100.33) (xy 175.26 100.33)
-		)
-		(stroke
-			(width 0)
-			(type default)
-		)
-	)
-	(wire
-		(pts
 			(xy 200.66 85.09) (xy 220.98 85.09)
 		)
@@
 		(pts
 			(xy 92.71 80.01) (xy 92.71 82.55)
-		)
-		(stroke
-			(width 0)
-			(type default)
-		)
-	)
-	(wire
-		(pts
-			(xy 163.83 85.09) (xy 171.45 85.09)
 		)
 		(stroke
@@
 	(hierarchical_label "PG"
 		(shape output)
-		(at 175.26 100.33 0)
+		(at 163.83 100.33 0)
 		(fields_autoplaced yes)
 		(effects
@@
 		(dnp no)
 		(fields_autoplaced yes)
-		(property "Reference" "R20"
+		(property "Reference" "R24"
 			(at 95.25 85.0899 0)
 			(effects
@@
 			(project "BasePower"
 				(path "/7a4c470e-f21a-4fdb-85db-575cfe7b758f/66a6072f-b93c-48b6-9ad2-cc693c587a24"
-					(reference "R20")
+					(reference "R24")
 					(unit 1)
 				)
@@
 		(dnp no)
 		(fields_autoplaced yes)
-		(property "Reference" "#PWR013"
+		(property "Reference" "#PWR014"
 			(at 128.27 118.11 0)
 			(effects
@@
 			(project "BasePower"
 				(path "/7a4c470e-f21a-4fdb-85db-575cfe7b758f/66a6072f-b93c-48b6-9ad2-cc693c587a24"
-					(reference "#PWR013")
+					(reference "#PWR014")
 					(unit 1)
 				)
@@
 	)
 	(symbol
-		(lib_id "Device:R_US")
-		(at 171.45 91.44 0)
-		(unit 1)
-		(exclude_from_sim no)
-		(in_bom yes)
-		(on_board yes)
-		(dnp no)
-		(fields_autoplaced yes)
-		(property "Reference" "R21"
-			(at 173.99 90.1699 0)
-			(effects
-				(font
-					(size 1.27 1.27)
-				)
-				(justify left)
-			)
-		)
-		(property "Value" "10kΩ"
-			(at 173.99 92.7099 0)
-			(effects
-				(font
-					(size 1.27 1.27)
-				)
-				(justify left)
-			)
-		)
-		(property "Footprint" "Resistor_SMD:R_0603_1608Metric"
-			(at 172.466 91.694 90)
-			(effects
-				(font
-					(size 1.27 1.27)
-				)
-				(hide yes)
-			)
-		)
-		(property "Datasheet" "~"
-			(at 171.45 91.44 0)
-			(effects
-				(font
-					(size 1.27 1.27)
-				)
-				(hide yes)
-			)
-		)
-		(property "Description" "Resistor, US symbol"
-			(at 171.45 91.44 0)
-			(effects
-				(font
-					(size 1.27 1.27)
-				)
-				(hide yes)
-			)
-		)
-		(pin "1"
-		)
-		(pin "2"
-		)
-		(instances
-			(project "BasePower"
-				(path "/7a4c470e-f21a-4fdb-85db-575cfe7b758f/66a6072f-b93c-48b6-9ad2-cc693c587a24"
-					(reference "R21")
-					(unit 1)
-				)
-			)
-		)
-	)
-	(symbol
 		(lib_id "Device:C_Small")
 		(at 77.47 95.25 0)
@@
 		(on_board yes)
 		(dnp no)
-		(property "Reference" "R23"
+		(property "Reference" "R26"
 			(at 95.25 100.3299 0)
 			(effects
@@
 			(project "BasePower"
 				(path "/7a4c470e-f21a-4fdb-85db-575cfe7b758f/66a6072f-b93c-48b6-9ad2-cc693c587a24"
-					(reference "R23")
+					(reference "R26")
 					(unit 1)
 				)
@@
 		(dnp no)
 		(fields_autoplaced yes)
-		(property "Reference" "R22"
+		(property "Reference" "R25"
 			(at 186.69 90.1699 0)
 			(effects
@@
 			(project "BasePower"
 				(path "/7a4c470e-f21a-4fdb-85db-575cfe7b758f/66a6072f-b93c-48b6-9ad2-cc693c587a24"
-					(reference "R22")
+					(reference "R25")
 					(unit 1)
 				)
@@
 		(on_board yes)
 		(dnp no)
-		(property "Reference" "R24"
+		(property "Reference" "R27"
 			(at 186.69 102.8699 0)
 			(effects
@@
 			(project "BasePower"
 				(path "/7a4c470e-f21a-4fdb-85db-575cfe7b758f/66a6072f-b93c-48b6-9ad2-cc693c587a24"
-					(reference "R24")
+					(reference "R27")
 					(unit 1)
 				)
