File: BatteryCharger/BatteryCharger.kicad_pcb (KiCad board)
At the start: 4 copper layers, 40 x 40 mm, 46 parts, among them J1 SYS, J2 ADAPTER, J3 BAT, J4 SMBus+STATUS, Q1 SiR638DP, Q2 SiR638DP, Q3 SiR500DP, Q4 BSC059N04LS6, Q5 SQJ868EP, U1 BQ24735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

Commit message: BatteryCharger board initially done
Parts:
- added J5: GND_BRIDGE, BW_PassiveMechanical:HolePad_2.5mm_3.5mm, F.Cu at (156.0, 117.5)
- added J6: GND_BRIDGE, BW_PassiveMechanical:HolePad_2.5mm_3.5mm, F.Cu at (144.5, 84.7)
- added REF**: BW_Logo_7.5x4.8mm, BW_Logo:BW_Logo_7.5x4.8mm, B.Cu at (139.2, 86.8)
- C12, C18, C2, D1, R1, R10, R12, R13, R4, R6, R8, R9, U2: moved to B.Cu
- moved R4 91.3 mm to (167.2, 95.7)
- moved D1 86.1 mm to (141.8, 107.0), turned to -90 degrees
- moved U2 84.4 mm to (138.2, 95.0), turned to 180 degrees
- moved R3 83.6 mm to (138.2, 108.8)
- moved C2 81.7 mm to (141.7, 99.7), turned to 180 degrees
- moved C11 77.9 mm to (138.2, 111.2), turned to 180 degrees
- moved C12 76.8 mm to (143.4, 103.4), turned to -90 degrees
- moved R1 70.1 mm to (141.8, 103.4), turned to 90 degrees
- moved C18 69.6 mm to (138.1, 97.6), turned to 180 degrees
- moved R6 68.2 mm to (135.4, 103.9), turned to 90 degrees
- moved R13 66.4 mm to (141.0, 97.0), turned to -90 degrees
- moved R9 65.7 mm to (133.8, 103.9), turned to -90 degrees
- moved R8 65.3 mm to (135.4, 100.8), turned to -90 degrees
- moved R12 63.2 mm to (137.0, 103.9), turned to 90 degrees
- moved R10 63.0 mm to (137.0, 100.8), turned to -90 degrees
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Routing:
- net Net-(D3-K): track 0.00 -> 58.0 mm
- net Net-(U1-BATDRV): track 0.00 -> 35.0 mm, vias 0 -> 1
- net Net-(U1-SRP): track 0.00 -> 30.0 mm, vias 0 -> 13
- net GND: track 0.00 -> 29.5 mm, vias 0 -> 36
- net Net-(J4-Pin_3): track 0.00 -> 23.7 mm, vias 0 -> 1
- net Net-(Q4-G): track 0.00 -> 21.4 mm
- net /SYS_PWR: track 0.00 -> 20.1 mm, vias 0 -> 48
- net Net-(J4-Pin_4): track 0.00 -> 19.7 mm, vias 0 -> 1
- net Net-(J4-Pin_2): track 0.00 -> 17.8 mm, vias 0 -> 1
- net Net-(J2-Pin_2): track 0.00 -> 17.3 mm, vias 0 -> 10
- net Net-(J4-Pin_1): track 0.00 -> 16.2 mm, vias 0 -> 1
- net Net-(Q1-G): track 0.00 -> 14.5 mm
- net Net-(Q4-S): track 0.00 -> 12.2 mm, vias 0 -> 31
- net Net-(Q2-D): track 0.00 -> 10.8 mm, vias 0 -> 9
- net +3.3V: track 0.00 -> 9.34 mm
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- added copper zone on B.Cu, net /SYS_PWR
- added copper zone on F.Cu, net /SYS_PWR
- added copper zone on B.Cu, net GND
- added copper zone on F.Cu, net GND
- added copper zone on In1.Cu, net GND
- added copper zone on In2.Cu, net GND
- added copper zone on F.Cu, net Net-(C1-Pad2)
- added copper zone on F.Cu, net Net-(D3-K)
- added copper zone on B.Cu, net Net-(J2-Pin_2)
- added copper zone on F.Cu, net Net-(J2-Pin_2)
- added copper zone on B.Cu, net Net-(Q2-D)
- added copper zone on F.Cu, net Net-(Q2-D)
- added copper zone on B.Cu, net Net-(Q4-S)
- added copper zone on F.Cu, net Net-(Q4-S)
- added copper zone on B.Cu, net Net-(U1-SRP)
- added copper zone on F.Cu, net Net-(U1-SRP)
Other:
- board text added: "19.5-24V"
- board text added: "<19V Li"
- board text added: "BAT±"
- board text added: "DC±"
- board text added: "Modular Audio Battery Charger"
- board text added: "SMBus"
- board text added: "SYS∓"
- board text added: "max 400W"

Commit message: BatteryCharger testing + small fix
U2 voltage source was incorrect
Connections:
- C1 pad 1: Net-(J2-Pin_2) -> /ADAPTER_IN
- C3 pad 1: Net-(J2-Pin_2) -> /ADAPTER_IN
- D1 pad 1: Net-(J2-Pin_2) -> /ADAPTER_IN
- J2 pad 2: Net-(J2-Pin_2) -> /ADAPTER_IN
- Q1 pad 5: Net-(J2-Pin_2) -> /ADAPTER_IN
- R3 pad 1: Net-(J2-Pin_2) -> /ADAPTER_IN
- R6 pad 1: Net-(J2-Pin_2) -> /ADAPTER_IN
- U2 pad 1: /SYS_PWR -> /ADAPTER_IN
Routing:
- net /ADAPTER_IN: track 0.00 -> 24.4 mm, vias 0 -> 10
- net Net-(J2-Pin_2): track 17.3 -> 0.00 mm, vias 10 -> 0
- net /SYS_PWR: track 20.1 -> 13.0 mm
- net GND: vias 36 -> 38
- added copper zone on B.Cu, net /ADAPTER_IN
- added copper zone on F.Cu, net /ADAPTER_IN
- removed copper zone on B.Cu, net Net-(J2-Pin_2)
- removed copper zone on F.Cu, net Net-(J2-Pin_2)
Other:
- board text added: "Modular Audio Battery Charger v1.1"
- board text removed: "Modular Audio Battery Charger"

Commit message: BatteryCharger v1.2: Increased input voltage range
Now 17.5V min instead of 19.5V min, to avoid power cycling at startup due to inrush
Parts:
- R6: value 287kΩ -> 210kΩ
- R8: value 432kΩ -> 64.9kΩ
- R9: value 40.2kΩ -> 28kΩ
Other:
- board text added: "17.5-24V"
- board text added: "Modular Audio Battery Charger v1.2"
- board text removed: "19.5-24V"
- board text removed: "Modular Audio Battery Charger v1.1"
